Commit message: ""

File: catkin_ws/src/franka_ros/franka_description/robots/common/franka_arm.xacro (robot description, xacro)
@@ -11,4 +11,7 @@
     params="arm_id:='panda' description_pkg:='franka_description' connected_to:='' xyz:='0 0 0' rpy:='0 0 0' gazebo:=false safety_distance:=0 joint_limits">
     <xacro:unless value="${not connected_to}">
+      <!-- <xacro:if value="${connected_to=='world'}">
+        <link name="${connected_to}" />
+      </xacro:if> -->
       <joint name="${arm_id}_joint_${connected_to}" type="fixed">
         <parent link="${connected_to}" />
