Commit message: it works now, but the base is no longer holonomic!

File: catkin_ws/src/franka_ros/franka_description/robots/common/franka_robot.xacro (robot description, xacro)
@@ -7,20 +7,8 @@
     <xacro:franka_arm arm_id="${arm_id}" safety_distance="0.03" gazebo="${gazebo}"
       joint_limits="${joint_limits}" connected_to="${parent}" xyz="${xyz}" rpy="${rpy}" />
-    <xacro:if value="${hand}">
-      <xacro:include filename="$(find franka_description)/robots/common/franka_hand.xacro" />
-      <xacro:franka_hand
-        arm_id="${arm_id}"
-        rpy="0 0 ${-pi/4}"
-        tcp_xyz="${tcp_xyz}"
-        tcp_rpy="${tcp_rpy}"
-        connected_to="${arm_id}_link8"
-        safety_distance="0.03"
-        gazebo="${gazebo}"
-      />
-    </xacro:if>
     <!-- Define additional Gazebo tags -->
     <xacro:if value="${gazebo}">
       <!-- PERHAPS COMMENT THIS OUT IT MIGHT BE DUPLICATING THE ROBOT GIVING THE FOLLOWING ERROR -->
-      <!-- Warning [Model.cc:216] Non-unique name[koala_joint7] detected 2 times in XML children of
+      <!-- Warning [Model.cc:216] Non-unique name[panda_joint7] detected 2 times in XML children of
       model with name[robot_b]. -->
       <xacro:if value="${parent != ''}">
@@ -35,32 +23,4 @@
         </joint>
       </xacro:if>
-      <xacro:gazebo-joint joint="${arm_id}_joint1"
-        transmission="hardware_interface/PositionJointInterface" />
-      <xacro:gazebo-joint joint="${arm_id}_joint2"
-        transmission="hardware_interface/PositionJointInterface" />
-      <xacro:gazebo-joint joint="${arm_id}_joint3"
-        transmission="hardware_interface/PositionJointInterface" />
-      <xacro:gazebo-joint joint="${arm_id}_joint4"
-        transmission="hardware_interface/PositionJointInterface" />
-      <xacro:gazebo-joint joint="${arm_id}_joint5"
-        transmission="hardware_interface/PositionJointInterface" />
-      <xacro:gazebo-joint joint="${arm_id}_joint6"
-        transmission="hardware_interface/PositionJointInterface" />
-      <xacro:gazebo-joint joint="${arm_id}_joint7"
-        transmission="hardware_interface/PositionJointInterface" />
-      <xacro:gazebo-joint joint="${arm_id}_joint1"
-        transmission="hardware_interface/VelocityJointInterface" />
-      <xacro:gazebo-joint joint="${arm_id}_joint2"
-        transmission="hardware_interface/VelocityJointInterface" />
-      <xacro:gazebo-joint joint="${arm_id}_joint3"
-        transmission="hardware_interface/VelocityJointInterface" />
-      <xacro:gazebo-joint joint="${arm_id}_joint4"
-        transmission="hardware_interface/VelocityJointInterface" />
-      <xacro:gazebo-joint joint="${arm_id}_joint5"
-        transmission="hardware_interface/VelocityJointInterface" />
-      <xacro:gazebo-joint joint="${arm_id}_joint6"
-        transmission="hardware_interface/VelocityJointInterface" />
-      <xacro:gazebo-joint joint="${arm_id}_joint7"
-        transmission="hardware_interface/VelocityJointInterface" />
       <xacro:gazebo-joint joint="${arm_id}_joint1"
         transmission="hardware_interface/EffortJointInterface" />
@@ -77,22 +37,8 @@
       <xacro:gazebo-joint joint="${arm_id}_joint7"
         transmission="hardware_interface/EffortJointInterface" />
-      <xacro:transmission-franka-state arm_id="${arm_id}" />
-      <xacro:transmission-franka-model arm_id="${arm_id}"
-        root="${arm_id}_joint1"
-        tip="${arm_id}_joint8"
-      />
-      <xacro:if value="${hand}">
-        <xacro:gazebo-joint joint="${arm_id}_finger_joint1"
-          transmission="hardware_interface/EffortJointInterface" />
-        <xacro:gazebo-joint joint="${arm_id}_finger_joint2"
-          transmission="hardware_interface/EffortJointInterface" />
-        <!-- Friction specific material for Rubber/Rubber contact -->
-        <xacro:gazebo-friction link="${arm_id}_leftfinger" mu="1.13" />
-        <xacro:gazebo-friction link="${arm_id}_rightfinger" mu="1.13" />
-      </xacro:if>
       <gazebo>
         <plugin name="gazebo_ros_control" filename="libgazebo_ros_control.so">
           <controlPeriod>0.001</controlPeriod>
-          <robotSimType>franka_gazebo/FrankaHWSim</robotSimType>
+          <robotSimType>gazebo_ros_control/DefaultRobotHWSim</robotSimType>
         </plugin>
         <self_collide>true</self_collide>

File: catkin_ws/src/franka_ros/franka_description/robots/common/utils.xacro (robot description, xacro)
@@ -2,6 +2,7 @@
 <robot xmlns:xacro="http://www.ros.org/wiki/xacro">
   <!-- Load inertial properties. Property is implicitly passed to macros. -->
-  <xacro:property name="inertial_config" value="$(find franka_description)/robots/common/inertial.yaml"/>
-  <xacro:property name="inertial" value="${xacro.load_yaml(inertial_config)}"/>
+  <xacro:property name="inertial_config"
+    value="$(find franka_description)/robots/common/inertial.yaml" />
+  <xacro:property name="inertial" value="${xacro.load_yaml(inertial_config)}" />
   <!-- ============================================================== -->
   <!-- Macro to add an <inertial> tag based on yaml-load properties   -->
@@ -11,15 +12,16 @@
   <!-- ============================================================== -->
   <xacro:macro name="inertial_props" params="name inertial:=^">
-      <xacro:unless value="${name in inertial}">${xacro.warning('No inertia properties defined for: ' + name)}</xacro:unless>
-      <xacro:if value="${name in inertial}">
-        <!-- Access inertia properties of link 'name' -->
-        <xacro:property name="inertial" value="${inertial[name]}" lazy_eval="false" />
-        <inertial>
-          <origin rpy="${inertial.origin.rpy}" xyz="${inertial.origin.xyz}" />
-          <mass value="${inertial.mass}" />
-          <xacro:property name="I" value="${inertial.inertia}" />
-          <inertia ixx="${I.xx}" ixy="${I.xy}" ixz="${I.xz}" iyy="${I.yy}" iyz="${I.yz}" izz="${I.zz}" />
-        </inertial>
-      </xacro:if>
+    <xacro:unless value="${name in inertial}">${xacro.warning('No inertia properties defined for: '
+      + name)}</xacro:unless>
+    <xacro:if value="${name in inertial}">
+      <!-- Access inertia properties of link 'name' -->
+      <xacro:property name="inertial" value="${inertial[name]}" lazy_eval="false" />
+      <inertial>
+        <origin rpy="${inertial.origin.rpy}" xyz="${inertial.origin.xyz}" />
+        <mass value="${inertial.mass}" />
+        <xacro:property name="I" value="${inertial.inertia}" />
+        <inertia ixx="${I.xx}" ixy="${I.xy}" ixz="${I.xz}" iyy="${I.yy}" iyz="${I.yz}" izz="${I.zz}" />
+      </inertial>
+    </xacro:if>
   </xacro:macro>
   <!-- ========================================================== -->
@@ -33,5 +35,6 @@
   <!-- self_collision_geometries:  self <collision> models        -->
   <!-- ========================================================== -->
-  <xacro:macro name="link_with_sc" params="name prefix=${arm_id}_ rpy:='0 0 0' **self_collision_geometries gazebo:=false">
+  <xacro:macro name="link_with_sc"
+    params="name prefix=${arm_id}_ rpy:='0 0 0' **self_collision_geometries gazebo:=false">
     <!-- sub-link defining detailed meshes for collision with environment -->
     <link name="${prefix}${name}">
@@ -86,5 +89,5 @@
     <xacro:property name="sz" value="${length / 2.0 if 'z' in direction else 0}" />
     <collision>
-      <origin xyz="${x} ${y} ${z}" rpy="${r} ${p} ${y}"/>
+      <origin xyz="${x} ${y} ${z}" rpy="${r} ${p} ${y}" />
       <geometry>
         <cylinder radius="${radius}" length="${length}" />
@@ -110,5 +113,6 @@
   <!-- transmission - type of the transmission of the joint       -->
   <!-- ========================================================== -->
-  <xacro:macro name="gazebo-joint" params="joint transmission:=hardware_interface/EffortJointInterface">
+  <xacro:macro name="gazebo-joint"
+    params="joint transmission:=hardware_interface/EffortJointInterface">
     <gazebo reference="${joint}">
       <!-- Needed for ODE to output external wrenches on joints -->
@@ -122,4 +126,5 @@
       <actuator name="${joint}_motor">
         <hardwareInterface>${transmission}</hardwareInterface>
+        <mechanicalReduction>1</mechanicalReduction>
       </actuator>
     </transmission>
@@ -145,5 +150,5 @@
             </ode>
           </friction>
-          <bounce/>
+          <bounce />
         </surface>
       </collision>
@@ -159,18 +164,46 @@
     <transmission name="${arm_id}_franka_state">
       <type>franka_hw/FrankaStateInterface</type>
-      <joint name="${arm_id}_joint1"><hardwareInterface>franka_hw/FrankaStateInterface</hardwareInterface></joint>
-      <joint name="${arm_id}_joint2"><hardwareInterface>franka_hw/FrankaStateInterface</hardwareInterface></joint>
-      <joint name="${arm_id}_joint3"><hardwareInterface>franka_hw/FrankaStateInterface</hardwareInterface></joint>
-      <joint name="${arm_id}_joint4"><hardwareInterface>franka_hw/FrankaStateInterface</hardwareInterface></joint>
-      <joint name="${arm_id}_joint5"><hardwareInterface>franka_hw/FrankaStateInterface</hardwareInterface></joint>
-      <joint name="${arm_id}_joint6"><hardwareInterface>franka_hw/FrankaStateInterface</hardwareInterface></joint>
-      <joint name="${arm_id}_joint7"><hardwareInterface>franka_hw/FrankaStateInterface</hardwareInterface></joint>
-      <actuator name="${arm_id}_motor1"><hardwareInterface>franka_hw/FrankaStateInterface</hardwareInterface></actuator>
-      <actuator name="${arm_id}_motor2"><hardwareInterface>franka_hw/FrankaStateInterface</hardwareInterface></actuator>
-      <actuator name="${arm_id}_motor3"><hardwareInterface>franka_hw/FrankaStateInterface</hardwareInterface></actuator>
-      <actuator name="${arm_id}_motor4"><hardwareInterface>franka_hw/FrankaStateInterface</hardwareInterface></actuator>
-      <actuator name="${arm_id}_motor5"><hardwareInterface>franka_hw/FrankaStateInterface</hardwareInterface></actuator>
-      <actuator name="${arm_id}_motor6"><hardwareInterface>franka_hw/FrankaStateInterface</hardwareInterface></actuator>
-      <actuator name="${arm_id}_motor7"><hardwareInterface>franka_hw/FrankaStateInterface</hardwareInterface></actuator>
+      <joint name="${arm_id}_joint1">
+        <hardwareInterface>franka_hw/FrankaStateInterface</hardwareInterface>
+      </joint>
+      <joint name="${arm_id}_joint2">
+        <hardwareInterface>franka_hw/FrankaStateInterface</hardwareInterface>
+      </joint>
+      <joint name="${arm_id}_joint3">
+        <hardwareInterface>franka_hw/FrankaStateInterface</hardwareInterface>
+      </joint>
+      <joint name="${arm_id}_joint4">
+        <hardwareInterface>franka_hw/FrankaStateInterface</hardwareInterface>
+      </joint>
+      <joint name="${arm_id}_joint5">
+        <hardwareInterface>franka_hw/FrankaStateInterface</hardwareInterface>
+      </joint>
+      <joint name="${arm_id}_joint6">
+        <hardwareInterface>franka_hw/FrankaStateInterface</hardwareInterface>
+      </joint>
+      <joint name="${arm_id}_joint7">
+        <hardwareInterface>franka_hw/FrankaStateInterface</hardwareInterface>
+      </joint>
+      <actuator name="${arm_id}_motor1">
+        <hardwareInterface>franka_hw/FrankaStateInterface</hardwareInterface>
+      </actuator>
+      <actuator name="${arm_id}_motor2">
+        <hardwareInterface>franka_hw/FrankaStateInterface</hardwareInterface>
+      </actuator>
+      <actuator name="${arm_id}_motor3">
+        <hardwareInterface>franka_hw/FrankaStateInterface</hardwareInterface>
+      </actuator>
+      <actuator name="${arm_id}_motor4">
+        <hardwareInterface>franka_hw/FrankaStateInterface</hardwareInterface>
+      </actuator>
+      <actuator name="${arm_id}_motor5">
+        <hardwareInterface>franka_hw/FrankaStateInterface</hardwareInterface>
+      </actuator>
+      <actuator name="${arm_id}_motor6">
+        <hardwareInterface>franka_hw/FrankaStateInterface</hardwareInterface>
+      </actuator>
+      <actuator name="${arm_id}_motor7">
+        <hardwareInterface>franka_hw/FrankaStateInterface</hardwareInterface>
+      </actuator>
     </transmission>
   </xacro:macro>
@@ -183,5 +216,6 @@
   <!-- tip    - Joint name of the tip of the robot (flange or hand) -->
   <!-- ============================================================ -->
-  <xacro:macro name="transmission-franka-model" params="arm_id:=panda root:=panda_joint1 tip:=panda_joint7">
+  <xacro:macro name="transmission-franka-model"
+    params="arm_id:=panda root:=panda_joint1 tip:=panda_joint7">
     <transmission name="${arm_id}_franka_model">
       <type>franka_hw/FrankaModelInterface</type>
@@ -194,6 +228,10 @@
         <hardwareInterface>franka_hw/FrankaModelInterface</hardwareInterface>
       </joint>
-      <actuator name="${root}_motor_root"><hardwareInterface>franka_hw/FrankaModelInterface</hardwareInterface></actuator>
-      <actuator name="${tip}_motor_tip"  ><hardwareInterface>franka_hw/FrankaModelInterface</hardwareInterface></actuator>
+      <actuator name="${root}_motor_root">
+        <hardwareInterface>franka_hw/FrankaModelInterface</hardwareInterface>
+      </actuator>
+      <actuator name="${tip}_motor_tip">
+        <hardwareInterface>franka_hw/FrankaModelInterface</hardwareInterface>
+      </actuator>
     </transmission>
   </xacro:macro>
@@ -201,7 +239,7 @@
     <inertial>
       <mass value="${mass}" />
-      <inertia ixx="${1./12 * mass * (3 * radius**2 + h**2)}" ixy = "0" ixz = "0"
-               iyy="${1./12 * mass * (3 * radius**2 + h**2)}" iyz = "0"
-               izz="${1./2  * mass * radius**2}" />
+      <inertia ixx="${1./12 * mass * (3 * radius**2 + h**2)}" ixy="0" ixz="0"
+        iyy="${1./12 * mass * (3 * radius**2 + h**2)}" iyz="0"
+        izz="${1./2  * mass * radius**2}" />
     </inertial>
   </xacro:macro>
@@ -214,13 +252,13 @@
   <!-- ========================================================================= -->
   <xacro:macro name="franka-limits" params="config name">
-      <xacro:property name="limits" value="${config[name]['limit']}" lazy_eval="false" />
-      <limit lower="${limits.lower}"
-             upper="${limits.upper}"
-             effort="${limits.effort}"
-             velocity="${limits.velocity}" />
-      <safety_controller k_position="100.0"
-                         k_velocity="40.0"
-                         soft_lower_limit="${limits.lower}"
-                         soft_upper_limit="${limits.upper}" />
+    <xacro:property name="limits" value="${config[name]['limit']}" lazy_eval="false" />
+    <limit lower="${limits.lower}"
+      upper="${limits.upper}"
+      effort="${limits.effort}"
+      velocity="${limits.velocity}" />
+    <safety_controller k_position="100.0"
+      k_velocity="40.0"
+      soft_lower_limit="${limits.lower}"
+      soft_upper_limit="${limits.upper}" />
   </xacro:macro>
 </robot>

File: catkin_ws/src/summit_xl_common/summit_xl_description/urdf/arms/franka/franka_robot.xacro (robot description, xacro)
@@ -7,16 +7,4 @@
     <xacro:franka_arm arm_id="${arm_id}" safety_distance="0.03" gazebo="${gazebo}"
       joint_limits="${joint_limits}" connected_to="${parent}" xyz="${xyz}" rpy="${rpy}" />
-    <xacro:if value="${hand}">
-      <xacro:include filename="$(find franka_description)/robots/common/franka_hand.xacro" />
-      <xacro:franka_hand
-        arm_id="${arm_id}"
-        rpy="0 0 ${-pi/4}"
-        tcp_xyz="${tcp_xyz}"
-        tcp_rpy="${tcp_rpy}"
-        connected_to="${arm_id}_link8"
-        safety_distance="0.03"
-        gazebo="${gazebo}"
-      />
-    </xacro:if>
     <!-- Define additional Gazebo tags -->
     <!-- <xacro:if value="${gazebo}"> -->
@@ -37,32 +25,4 @@
       </xacro:if> -->
       <xacro:gazebo-joint joint="${arm_id}_joint1"
-        transmission="hardware_interface/PositionJointInterface" />
-      <xacro:gazebo-joint joint="${arm_id}_joint2"
-        transmission="hardware_interface/PositionJointInterface" />
-      <xacro:gazebo-joint joint="${arm_id}_joint3"
-        transmission="hardware_interface/PositionJointInterface" />
-      <xacro:gazebo-joint joint="${arm_id}_joint4"
-        transmission="hardware_interface/PositionJointInterface" />
-      <xacro:gazebo-joint joint="${arm_id}_joint5"
-        transmission="hardware_interface/PositionJointInterface" />
-      <xacro:gazebo-joint joint="${arm_id}_joint6"
-        transmission="hardware_interface/PositionJointInterface" />
-      <xacro:gazebo-joint joint="${arm_id}_joint7"
-        transmission="hardware_interface/PositionJointInterface" />
-      <xacro:gazebo-joint joint="${arm_id}_joint1"
-        transmission="hardware_interface/VelocityJointInterface" />
-      <xacro:gazebo-joint joint="${arm_id}_joint2"
-        transmission="hardware_interface/VelocityJointInterface" />
-      <xacro:gazebo-joint joint="${arm_id}_joint3"
-        transmission="hardware_interface/VelocityJointInterface" />
-      <xacro:gazebo-joint joint="${arm_id}_joint4"
-        transmission="hardware_interface/VelocityJointInterface" />
-      <xacro:gazebo-joint joint="${arm_id}_joint5"
-        transmission="hardware_interface/VelocityJointInterface" />
-      <xacro:gazebo-joint joint="${arm_id}_joint6"
-        transmission="hardware_interface/VelocityJointInterface" />
-      <xacro:gazebo-joint joint="${arm_id}_joint7"
-        transmission="hardware_interface/VelocityJointInterface" />
-      <xacro:gazebo-joint joint="${arm_id}_joint1"
         transmission="hardware_interface/EffortJointInterface" />
       <xacro:gazebo-joint joint="${arm_id}_joint2"
@@ -78,22 +38,8 @@
       <xacro:gazebo-joint joint="${arm_id}_joint7"
         transmission="hardware_interface/EffortJointInterface" />
-      <xacro:transmission-franka-state arm_id="${arm_id}" />
-      <xacro:transmission-franka-model arm_id="${arm_id}"
-        root="${arm_id}_joint1"
-        tip="${arm_id}_joint8"
-      />
-      <xacro:if value="${hand}">
-        <xacro:gazebo-joint joint="${arm_id}_finger_joint1"
-          transmission="hardware_interface/EffortJointInterface" />
-        <xacro:gazebo-joint joint="${arm_id}_finger_joint2"
-          transmission="hardware_interface/EffortJointInterface" />
-        <!-- Friction specific material for Rubber/Rubber contact -->
-        <xacro:gazebo-friction link="${arm_id}_leftfinger" mu="1.13" />
-        <xacro:gazebo-friction link="${arm_id}_rightfinger" mu="1.13" />
-      </xacro:if>
       <gazebo>
         <plugin name="gazebo_ros_control" filename="libgazebo_ros_control.so">
           <controlPeriod>0.001</controlPeriod>
-          <robotSimType>franka_gazebo/FrankaHWSim</robotSimType>
+          <robotSimType>gazebo_ros_control/DefaultRobotHWSim</robotSimType>
         </plugin>
         <self_collide>true</self_collide>

File: catkin_ws/src/summit_xl_common/summit_xl_description/urdf/wheels/omni_wheel.urdf.xacro (robot description, xacro)
@@ -7,16 +7,16 @@
   <xacro:property name="omni_wheel_mass" value="6.5" /> <!-- in kg-->
   <xacro:macro name="cylinder_inertia" params="m r h">
-    <inertia  ixx="${m*(3*r*r+h*h)/12}" ixy = "0" ixz = "0"
-              iyy="${m*r*r/2}" iyz = "0"
-              izz="${m*(3*r*r+h*h)/12}" />
+    <inertia ixx="${m*(3*r*r+h*h)/12}" ixy="0" ixz="0"
+      iyy="${m*r*r/2}" iyz="0"
+      izz="${m*(3*r*r+h*h)/12}" />
   </xacro:macro>
   <xacro:macro name="omni_wheel" params="prefix parent *origin reflect hq">
     <joint name="${prefix}_wheel_joint" type="continuous">
-      <parent link="${parent}"/>
-      <child link="${prefix}_wheel_link"/>
+      <parent link="${parent}" />
+      <child link="${prefix}_wheel_link" />
       <xacro:insert_block name="origin" />
       <axis xyz="0 1 0" rpy="0 0 0" />
-      <limit effort="100" velocity="100"/>
-      <joint_properties damping="0.0" friction="0.0"/>
+      <limit effort="100" velocity="100" />
+      <joint_properties damping="0.0" friction="0.0" />
     </joint>
     <link name="${prefix}_wheel_link">
@@ -33,5 +33,5 @@
               <mesh filename="package://summit_xl_description/meshes/wheels/omni_wheel_2.dae" />
             </geometry>
-		  </xacro:unless>
+          </xacro:unless>
         </xacro:if>
         <xacro:unless value="${hq}">
@@ -42,12 +42,13 @@
         </xacro:unless>
         <material name="darkgrey">
-           <color rgba="0.2 0.2 0.2 1"/>
+          <color rgba="0.2 0.2 0.2 1" />
         </material>
       </visual>
       <collision>
-				<origin xyz="0 0 0" rpy="${PI/2} 0 0" />
+        <origin xyz="0 0 0" rpy="${PI/2} 0 0" />
         <geometry>
-          <!--sphere radius="${omni_wheel_radius}" /-->
-<!--
+          <!--sphere
+          radius="${omni_wheel_radius}" /-->
+          <!--
           <xacro:if value="${reflect}">
               <mesh filename="package://summit_xl_description/meshes/wheels/omni_wheel_1.dae" />
@@ -57,6 +58,6 @@
 					</xacro:unless>
 -->
-					<cylinder length="${omni_wheel_height}" radius="${omni_wheel_radius}" />
-					<!-- sphere radius="${omni_wheel_radius}"/-->
+          <cylinder length="${omni_wheel_height}" radius="${omni_wheel_radius}" />
+          <!-- sphere radius="${omni_wheel_radius}"/-->
         </geometry>
       </collision>
@@ -64,24 +65,26 @@
         <mass value="${omni_wheel_mass}" />
         <origin xyz="0 0 0" />
-        <xacro:cylinder_inertia  m="${omni_wheel_mass}" r="${omni_wheel_radius}" h="${omni_wheel_height}" />
+        <xacro:cylinder_inertia m="${omni_wheel_mass}" r="${omni_wheel_radius}"
+          h="${omni_wheel_height}" />
       </inertial>
     </link>
-    <!-- Transmission is important to link the joints and the controller (see summit_xl_control/config/summit_xl_control.yaml)-->
+    <!-- Transmission is important to link the joints and the controller (see
+    summit_xl_control/config/summit_xl_control.yaml)-->
     <transmission name="${prefix}_wheel_joint_trans">
       <type>transmission_interface/SimpleTransmission</type>
-      <joint name="${prefix}_wheel_joint" >
+      <joint name="${prefix}_wheel_joint">
         <hardwareInterface>hardware_interface/VelocityJointInterface</hardwareInterface>
       </joint>
       <actuator name="${prefix}_wheel_joint_motor">
-         <mechanicalReduction>1</mechanicalReduction>
+        <mechanicalReduction>1</mechanicalReduction>
       </actuator>
     </transmission>
     <gazebo reference="${prefix}_wheel_link">
-		<mu1 value="0.0"/>
-		<mu2 value="0.0"/>
-		<kp value="10000000.0" />
-		<kd value="1.0" />
-		<fdir1 value="1 0 0"/>
-        <turnGravityOff>false</turnGravityOff>
+      <mu1 value="10.0" />
+      <mu2 value="10.0" />
+      <kp value="10000000.0" />
+      <kd value="1.0" />
+      <fdir1 value="1 0 0" />
+      <turnGravityOff>false</turnGravityOff>
     </gazebo>
   </xacro:macro>
