Commit message: it works now, but the base is no longer holonomic

File: catkin_ws/src/franka_ros/franka_description/robots/panda/panda.urdf (robot description, URDF)
Before this commit: robot panda, 17 links, 17 joints
Links:
- added link world
- link panda_link0: mass None -> 0.629769
- link panda_link0_sc: geometry 
- link panda_link1: mass None -> 4.970684
- link panda_link1_sc: geometry 
- link panda_link2: mass None -> 0.646926
- link panda_link2_sc: geometry 
- link panda_link3: mass None -> 3.228604
- link panda_link3_sc: geometry 
- link panda_link4: mass None -> 3.587895
- link panda_link4_sc: geometry 
- link panda_link5: mass None -> 1.225946
- link panda_link5_sc: geometry 
- link panda_link6: mass None -> 1.666555
- link panda_link6_sc: geometry 
- link panda_link7: mass None -> 0.735522
- link panda_link7_sc: geometry 
Joints:
- added joint world_joint: type fixed, parent world, child panda_link0, origin xyz=10 10 0 rpy=0 0 0

File: catkin_ws/src/franka_ros/franka_description/robots/panda/panda.urdf.xacro (robot description, xacro)
@@ -12,5 +12,5 @@
   <xacro:arg name="tcp_rpy" default="0 0 0" />
   <!-- Is the robot being simulated in gazebo?" -->
-  <xacro:arg name="gazebo" default="false" />
+  <xacro:arg name="gazebo" default="true" />
   <!-- If `gazebo` arg is set, to which frame shall $(arm_id)_link0 be parented. Empty string for
   not fixing at all -->
