Commit message: generated a moveit package for the panda with the right controller

File: catkin_ws/src/summit_xl_common/moveit/panda_moveit_config/config/gazebo_summit_xl.urdf (robot description, URDF)
Before this commit: robot summit_xl, 39 links, 38 joints
Links:
- removed link summit_xl__link0
- removed link summit_xl__link0_sc
- removed link summit_xl__link1
- removed link summit_xl__link1_sc
- removed link summit_xl__link2
- removed link summit_xl__link2_sc
- removed link summit_xl__link3
- removed link summit_xl__link3_sc
- removed link summit_xl__link4
- removed link summit_xl__link4_sc
- removed link summit_xl__link5
- removed link summit_xl__link5_sc
- removed link summit_xl__link6
- removed link summit_xl__link6_sc
- removed link summit_xl__link7
- removed link summit_xl__link7_sc
- removed link summit_xl__link8
- added link panda_link0, mass 0.629769; collision mesh filename=package://franka_description/meshes/collision/link0.stl; visual mesh filename=package://franka_description/meshes/visual/link0.dae
- added link panda_link0_sc
- added link panda_link1, mass 4.970684; collision mesh filename=package://franka_description/meshes/collision/link1.stl; visual mesh filename=package://franka_description/meshes/visual/link1.dae
- added link panda_link1_sc
- added link panda_link2, mass 0.646926; collision mesh filename=package://franka_description/meshes/collision/link2.stl; visual mesh filename=package://franka_description/meshes/visual/link2.dae
- added link panda_link2_sc
- added link panda_link3, mass 3.228604; collision mesh filename=package://franka_description/meshes/collision/link3.stl; visual mesh filename=package://franka_description/meshes/visual/link3.dae
- added link panda_link3_sc
- added link panda_link4, mass 3.587895; collision mesh filename=package://franka_description/meshes/collision/link4.stl; visual mesh filename=package://franka_description/meshes/visual/link4.dae
- added link panda_link4_sc
- added link panda_link5, mass 1.225946; collision mesh filename=package://franka_description/meshes/collision/link5.stl; visual mesh filename=package://franka_description/meshes/visual/link5.dae
- added link panda_link5_sc
- added link panda_link6, mass 1.666555; collision mesh filename=package://franka_description/meshes/collision/link6.stl; visual mesh filename=package://franka_description/meshes/visual/link6.dae
- added link panda_link6_sc
- added link panda_link7, mass 0.735522; collision mesh filename=package://franka_description/meshes/collision/link7.stl; visual mesh filename=package://franka_description/meshes/visual/link7.dae
- added link panda_link7_sc
- added link panda_link8
Joints:
- removed joint summit_xl__joint1
- removed joint summit_xl__joint2
- removed joint summit_xl__joint3
- removed joint summit_xl__joint4
- removed joint summit_xl__joint5
- removed joint summit_xl__joint6
- removed joint summit_xl__joint7
- removed joint summit_xl__joint8
- removed joint summit_xl__joint_summit_xl_base_link
- removed joint summit_xl__link0_sc_joint
- removed joint summit_xl__link1_sc_joint
- removed joint summit_xl__link2_sc_joint
- removed joint summit_xl__link3_sc_joint
- removed joint summit_xl__link4_sc_joint
- removed joint summit_xl__link5_sc_joint
- removed joint summit_xl__link6_sc_joint
- removed joint summit_xl__link7_sc_joint
- added joint panda_joint1: type revolute, parent panda_link0, child panda_link1, origin xyz=0 0 0.333 rpy=0 0 0, axis 0 0 1, limit lower=-2.8973 upper=2.8973 effort=87.0 velocity=2.175
- added joint panda_joint2: type revolute, parent panda_link1, child panda_link2, origin xyz=0 0 0 rpy=-1.5707963267948966 0 0, axis 0 0 1, limit lower=-1.7628 upper=1.7628 effort=87.0 velocity=2.175
- added joint panda_joint3: type revolute, parent panda_link2, child panda_link3, origin xyz=0 -0.316 0 rpy=1.5707963267948966 0 0, axis 0 0 1, limit lower=-2.8973 upper=2.8973 effort=87.0 velocity=2.175
- added joint panda_joint4: type revolute, parent panda_link3, child panda_link4, origin xyz=0.0825 0 0 rpy=1.5707963267948966 0 0, axis 0 0 1, limit lower=-3.0718 upper=-0.0698 effort=87.0 velocity=2.175
- added joint panda_joint5: type revolute, parent panda_link4, child panda_link5, origin xyz=-0.0825 0.384 0 rpy=-1.5707963267948966 0 0, axis 0 0 1, limit lower=-2.8973 upper=2.8973 effort=12.0 velocity=2.61
- added joint panda_joint6: type revolute, parent panda_link5, child panda_link6, origin xyz=0 0 0 rpy=1.5707963267948966 0 0, axis 0 0 1, limit lower=-0.0175 upper=3.7525 effort=12.0 velocity=2.61
- added joint panda_joint7: type revolute, parent panda_link6, child panda_link7, origin xyz=0.088 0 0 rpy=1.5707963267948966 0 0, axis 0 0 1, limit lower=-2.8973 upper=2.8973 effort=12.0 velocity=2.61
- added joint panda_joint8: type fixed, parent panda_link7, child panda_link8, origin xyz=0 0 0.107 rpy=0 0 0
- added joint panda_joint_summit_xl_base_link: type fixed, parent summit_xl_base_link, child panda_link0, origin xyz=0.2 -0.15 0.380 rpy=0 0 0
- added joint panda_link0_sc_joint: type fixed, parent panda_link0, child panda_link0_sc, origin rpy=0 0 0
- added joint panda_link1_sc_joint: type fixed, parent panda_link1, child panda_link1_sc, origin rpy=0 0 0
- added joint panda_link2_sc_joint: type fixed, parent panda_link2, child panda_link2_sc, origin rpy=0 0 0
- added joint panda_link3_sc_joint: type fixed, parent panda_link3, child panda_link3_sc, origin rpy=0 0 0
- added joint panda_link4_sc_joint: type fixed, parent panda_link4, child panda_link4_sc, origin rpy=0 0 0
- added joint panda_link5_sc_joint: type fixed, parent panda_link5, child panda_link5_sc, origin rpy=0 0 0
- added joint panda_link6_sc_joint: type fixed, parent panda_link6, child panda_link6_sc, origin rpy=0 0 0
- added joint panda_link7_sc_joint: type fixed, parent panda_link7, child panda_link7_sc, origin rpy=0 0 0.7853981633974483
