Commit message: changed some stuff so that the panda controllers can run

File: catkin_ws/src/summit_xl_common/summit_xl_description/robots/summit_xls_panda.urdf.xacro (robot description, xacro)
@@ -54,5 +54,5 @@
 	<xacro:property name="arm_offset_yaw" value="0.0" />
 	<!-- Name for this robot -->
-	<xacro:arg name="arm_id" default="heyo" />
+	<xacro:arg name="arm_id" default="panda" />
 	<!-- Should a franka_gripper be mounted at the flange?" -->
 	<xacro:arg name="hand" default="false" />
@@ -80,4 +80,5 @@
 	<xacro:arg name="ros_planar_move_plugin_force_based" default="false" />
 	<xacro:arg name="gpu" default="false" />
+	<xacro:arg name="arm_id" default="panda" />
 	<xacro:macro name="summit_xl" params="prefix publish_bf hq">
 		<!-- *************** -->
@@ -149,5 +150,5 @@
 		</joint> -->
 		<!-- <xacro:vx300s base_parent="$(arg prefix)arm_base_link" prefix="$(arg prefix)arm_" /> -->
-		<xacro:franka_robot arm_id="$(arg prefix)"
+		<xacro:franka_robot arm_id="$(arg arm_id)"
 			joint_limits="${xacro.load_yaml('$(find franka_description)/robots/panda/joint_limits.yaml')}"
 			hand="$(arg hand)"
@@ -165,5 +166,5 @@
 		</xacro:sensor_intel_d435> -->
 	</xacro:macro>
-	<xacro:ros_control />
+	<!-- <xacro:ros_control /> -->
 	<xacro:if value="$(arg ros_planar_move_plugin)">
 		<xacro:omni_steering prefix="$(arg prefix)" publish_tf="true"

File: catkin_ws/src/summit_xl_common/summit_xl_description/robots/summit_xls_std.urdf.xacro (robot description, xacro)
@@ -4,5 +4,6 @@
 	<!-- Imported elements -->
 	<!-- ***************** -->
-	<!-- First we import all posible elements defined in the urdf.xacro files. All these elements are defined as macro:xacros -->
+	<!-- First we import all posible elements defined in the urdf.xacro files. All these elements
+	are defined as macro:xacros -->
 	<!-- Import summit XL base elements -->
 	<xacro:include filename="$(find summit_xl_description)/urdf/bases/summit_xls_base.urdf.xacro" />
@@ -10,87 +11,108 @@
 	<xacro:include filename="$(find summit_xl_description)/urdf/wheels/omni_wheel.urdf.xacro" />
 	<xacro:include filename="$(find summit_xl_description)/urdf/wheels/rubber_wheel.urdf.xacro" />
-	<xacro:include filename="$(find summit_xl_description)/urdf/structures/structure_hokuyo.urdf.xacro" />
+	<xacro:include
+		filename="$(find summit_xl_description)/urdf/structures/structure_hokuyo.urdf.xacro" />
 	<!-- Import all available sensors -->
 	<xacro:include filename="$(find robotnik_sensors)/urdf/all_sensors.urdf.xacro" />
-	<xacro:property name="PI" value="3.1415926535897931"/>
+	<xacro:property name="PI" value="3.1415926535897931" />
 	<!-- Wheel parameters -->
 	<!-- Wheel parameters -->
-	<xacro:property name="wheel_offset_x" value="0.2225" />    <!-- x,y,z in translation from base_link to the center of the wheel -->
+	<xacro:property name="wheel_offset_x" value="0.2225" />    <!-- x,y,z in translation from base_link
+	to the center of the wheel -->
 	<xacro:property name="wheel_offset_y" value="0.2045" />
 	<xacro:property name="wheel_offset_z" value="0.0" />
-	<xacro:property name="front_laser_offset_x" value="0.2865"/>
-	<xacro:property name="front_laser_offset_y" value="-0.20894"/>
-	<xacro:property name="front_laser_offset_z" value="0.2973"/>
-	<xacro:property name="rear_laser_offset_x" value="-0.2865"/>
-	<xacro:property name="rear_laser_offset_y" value="0.20894"/>
-	<xacro:property name="rear_laser_offset_z" value="0.2973"/>
-	<xacro:property name="front_ptz_camera_offset_x" value="0.308"/>
-	<xacro:property name="front_ptz_camera_offset_y" value="0.141"/>
-	<xacro:property name="front_ptz_camera_offset_z" value="0.195"/>
-	<xacro:property name="rear_ptz_camera_offset_x" value="-0.308"/>
-	<xacro:property name="rear_ptz_camera_offset_y" value="-0.141"/>
-	<xacro:property name="rear_ptz_camera_offset_z" value="0.195"/>
-	<xacro:property name="imu_offset_x" value="0.127"/>
-	<xacro:property name="imu_offset_y" value="-0.129"/>
-	<xacro:property name="imu_offset_z" value="0.212"/>
-	<xacro:property name="front_rgbd_camera_offset_x" value="0.35850"/>
-	<xacro:property name="front_rgbd_camera_offset_y" value="0.0"/>
-	<xacro:property name="front_rgbd_camera_offset_z" value="0.25062"/>
-	<xacro:property name="gps_offset_x" value="-0.365"/>
-	<xacro:property name="gps_offset_y" value="-0.167"/>
-	<xacro:property name="gps_offset_z" value="0.302"/>
+	<xacro:property name="front_laser_offset_x" value="0.2865" />
+	<xacro:property name="front_laser_offset_y" value="-0.20894" />
+	<xacro:property name="front_laser_offset_z" value="0.2973" />
+	<xacro:property name="rear_laser_offset_x" value="-0.2865" />
+	<xacro:property name="rear_laser_offset_y" value="0.20894" />
+	<xacro:property name="rear_laser_offset_z" value="0.2973" />
+	<xacro:property name="front_ptz_camera_offset_x" value="0.308" />
+	<xacro:property name="front_ptz_camera_offset_y" value="0.141" />
+	<xacro:property name="front_ptz_camera_offset_z" value="0.195" />
+	<xacro:property name="rear_ptz_camera_offset_x" value="-0.308" />
+	<xacro:property name="rear_ptz_camera_offset_y" value="-0.141" />
+	<xacro:property name="rear_ptz_camera_offset_z" value="0.195" />
+	<xacro:property name="imu_offset_x" value="0.127" />
+	<xacro:property name="imu_offset_y" value="-0.129" />
+	<xacro:property name="imu_offset_z" value="0.212" />
+	<xacro:property name="front_rgbd_camera_offset_x" value="0.35850" />
+	<xacro:property name="front_rgbd_camera_offset_y" value="0.0" />
+	<xacro:property name="front_rgbd_camera_offset_z" value="0.25062" />
+	<xacro:property name="gps_offset_x" value="-0.365" />
+	<xacro:property name="gps_offset_y" value="-0.167" />
+	<xacro:property name="gps_offset_z" value="0.302" />
 	<!-- Flag to select the high or low quality model -->
 	<xacro:property name="hq" value="true" />
-	<xacro:arg name="prefix" default="summit_xl_"/>
-	<xacro:arg name="ros_planar_move_plugin" default="false"/>
-	<xacro:arg name="ros_planar_move_plugin_force_based" default="false"/>
-	<xacro:arg name="gpu" default="false"/>
-    <xacro:macro name="summit_xl" params="prefix publish_bf hq">
+	<xacro:arg name="prefix" default="summit_xl_" />
+	<xacro:arg name="ros_planar_move_plugin" default="false" />
+	<xacro:arg name="ros_planar_move_plugin_force_based" default="false" />
+	<xacro:arg name="gpu" default="false" />
+	<xacro:macro name="summit_xl" params="prefix publish_bf hq">
 		<!-- *************** -->
 		<!-- Robots Elements -->
 		<!-- *************** -->
-		<!-- Here we create the robot elements using the xacro:macros imported at the beggining of this file -->
+		<!-- Here we create the robot elements using the xacro:macros imported at the beggining of
+		this file -->
 		<!-- Summit XL base -->
 		<xacro:summit_xls_base prefix="$(arg prefix)" publish_bf="true" hq="${hq}" />
-		<xacro:omni_wheel prefix="$(arg prefix)front_right" parent="$(arg prefix)base_link" reflect="false" hq="${hq}">
-			<origin xyz="${wheel_offset_x} -${wheel_offset_y} ${wheel_offset_z}" rpy="0 0 0"/>
+		<xacro:omni_wheel prefix="$(arg prefix)front_right" parent="$(arg prefix)base_link"
+			reflect="false" hq="${hq}">
+			<origin xyz="${wheel_offset_x} -${wheel_offset_y} ${wheel_offset_z}" rpy="0 0 0" />
 		</xacro:omni_wheel>
-		<xacro:omni_wheel prefix="$(arg prefix)front_left" parent="$(arg prefix)base_link" reflect="true" hq="${hq}">
-			<origin xyz="${wheel_offset_x} ${wheel_offset_y} ${wheel_offset_z}" rpy="0 0 0"/>
+		<xacro:omni_wheel prefix="$(arg prefix)front_left" parent="$(arg prefix)base_link"
+			reflect="true" hq="${hq}">
+			<origin xyz="${wheel_offset_x} ${wheel_offset_y} ${wheel_offset_z}" rpy="0 0 0" />
 		</xacro:omni_wheel>
-		<xacro:omni_wheel prefix="$(arg prefix)back_left" parent="$(arg prefix)base_link" reflect="true" hq="${hq}">
-			<origin xyz="-${wheel_offset_x} ${wheel_offset_y} ${wheel_offset_z}" rpy="0 0 0"/>
+		<xacro:omni_wheel prefix="$(arg prefix)back_left" parent="$(arg prefix)base_link"
+			reflect="true" hq="${hq}">
+			<origin xyz="-${wheel_offset_x} ${wheel_offset_y} ${wheel_offset_z}" rpy="0 0 0" />
 		</xacro:omni_wheel>
-		<xacro:omni_wheel prefix="$(arg prefix)back_right" parent="$(arg prefix)base_link" reflect="false" hq="${hq}">
-			<origin xyz="-${wheel_offset_x} -${wheel_offset_y} ${wheel_offset_z}" rpy="0 0 0"/>
+		<xacro:omni_wheel prefix="$(arg prefix)back_right" parent="$(arg prefix)base_link"
+			reflect="false" hq="${hq}">
+			<origin xyz="-${wheel_offset_x} -${wheel_offset_y} ${wheel_offset_z}" rpy="0 0 0" />
 		</xacro:omni_wheel>
-        <!-- IMU -->
-		<xacro:sensor_imu prefix="$(arg prefix)imu" parent="$(arg prefix)base_link" topic="imu/data_raw">
-			<origin xyz="${imu_offset_x} ${imu_offset_y} ${imu_offset_z}" rpy="0 0 0"/>
+		<!-- IMU -->
+		<xacro:sensor_imu prefix="$(arg prefix)imu" parent="$(arg prefix)base_link"
+			topic="imu/data_raw">
+			<origin xyz="${imu_offset_x} ${imu_offset_y} ${imu_offset_z}" rpy="0 0 0" />
 		</xacro:sensor_imu>
 		<!-- SENSORS -->
-		<xacro:sensor_sick_s300 prefix="$(arg prefix)front_laser" parent="$(arg prefix)base_link" prefix_topic="front_laser" gpu="$(arg gpu)">
-			<origin xyz="${front_laser_offset_x} ${front_laser_offset_y} ${front_laser_offset_z}" rpy="0 ${-PI} ${3/4*PI}" />
+		<xacro:sensor_sick_s300 prefix="$(arg prefix)front_laser" parent="$(arg prefix)base_link"
+			prefix_topic="front_laser" gpu="$(arg gpu)">
+			<origin xyz="${front_laser_offset_x} ${front_laser_offset_y} ${front_laser_offset_z}"
+				rpy="0 ${-PI} ${3/4*PI}" />
 		</xacro:sensor_sick_s300>
-		<xacro:sensor_sick_s300 prefix="$(arg prefix)rear_laser" parent="$(arg prefix)base_link" prefix_topic="rear_laser" gpu="$(arg gpu)">
-			<origin xyz="${rear_laser_offset_x} ${rear_laser_offset_y} ${rear_laser_offset_z}" rpy="0 ${-PI} ${-1/4*PI}" />
+		<xacro:sensor_sick_s300 prefix="$(arg prefix)rear_laser" parent="$(arg prefix)base_link"
+			prefix_topic="rear_laser" gpu="$(arg gpu)">
+			<origin xyz="${rear_laser_offset_x} ${rear_laser_offset_y} ${rear_laser_offset_z}"
+				rpy="0 ${-PI} ${-1/4*PI}" />
 		</xacro:sensor_sick_s300>
-		<!--xacro:sensor_axis_m5013 prefix="$(arg prefix)front_ptz_camera" parent="$(arg prefix)base_link">
-			<origin xyz="${front_ptz_camera_offset_x} ${front_ptz_camera_offset_y} ${front_ptz_camera_offset_z}" rpy="${-PI/2} 0 0"/>
+		<!--xacro:sensor_axis_m5013
+		prefix="$(arg prefix)front_ptz_camera" parent="$(arg prefix)base_link">
+			<origin xyz="${front_ptz_camera_offset_x} ${front_ptz_camera_offset_y}
+		${front_ptz_camera_offset_z}" rpy="${-PI/2} 0 0"/>
 		</xacro:sensor_axis_m5013-->
-		<!--xacro:sensor_axis_m5013 prefix="$(arg prefix)rear_ptz_camera" parent="$(arg prefix)base_link">
-			<origin xyz="${rear_ptz_camera_offset_x} ${rear_ptz_camera_offset_y} ${rear_ptz_camera_offset_z}" rpy="${-PI/2} 0 ${PI}"/>
+		<!--xacro:sensor_axis_m5013
+		prefix="$(arg prefix)rear_ptz_camera" parent="$(arg prefix)base_link">
+			<origin xyz="${rear_ptz_camera_offset_x} ${rear_ptz_camera_offset_y} ${rear_ptz_camera_offset_z}"
+		rpy="${-PI/2} 0 ${PI}"/>
 		</xacro:sensor_axis_m5013-->
-		<xacro:sensor_orbbec_astra prefix="$(arg prefix)front_rgbd_camera" parent="$(arg prefix)base_link" prefix_topic="front_rgbd_camera">
-			<origin xyz="${front_rgbd_camera_offset_x} ${front_rgbd_camera_offset_y} ${front_rgbd_camera_offset_z}" rpy="0 0 0"/>
+		<xacro:sensor_orbbec_astra prefix="$(arg prefix)front_rgbd_camera"
+			parent="$(arg prefix)base_link" prefix_topic="front_rgbd_camera">
+			<origin
+				xyz="${front_rgbd_camera_offset_x} ${front_rgbd_camera_offset_y} ${front_rgbd_camera_offset_z}"
+				rpy="0 0 0" />
 		</xacro:sensor_orbbec_astra>
-		<!--xacro:sensor_gps prefix="$(arg prefix)gps" parent="$(arg prefix)base_link">
+		<!--xacro:sensor_gps
+		prefix="$(arg prefix)gps" parent="$(arg prefix)base_link">
 			<origin xyz="${gps_offset_x} ${gps_offset_y} ${gps_offset_z}" rpy="0 0 0"/>
 		</xacro:sensor_gps-->
-   </xacro:macro>
-   <xacro:ros_control/>
-   <xacro:if value="$(arg ros_planar_move_plugin)">
-	   <xacro:omni_steering prefix="$(arg prefix)" publish_tf="true" force_based="$(arg ros_planar_move_plugin_force_based)"/>
-   </xacro:if>
-   <xacro:summit_xl prefix="$(arg prefix)" publish_bf="true" hq="true"/>
+	</xacro:macro>
+	<xacro:ros_control />
+	<xacro:if value="$(arg ros_planar_move_plugin)">
+		<xacro:omni_steering prefix="$(arg prefix)" publish_tf="true"
+			force_based="$(arg ros_planar_move_plugin_force_based)" />
+	</xacro:if>
+	<xacro:summit_xl prefix="$(arg prefix)" publish_bf="true" hq="true" />
 </robot>

Commit message: Added Caspers navigation code

File: catkin_ws/src/summit_xl_common/summit_xl_description/robots/summit_xls_panda.urdf.xacro (robot description, xacro)
@@ -8,4 +8,23 @@
 	<!-- Import summit XL base elements -->
 	<xacro:include filename="$(find summit_xl_description)/urdf/bases/summit_xls_base.urdf.xacro" />
+	<!-- Define the joint between world and base_footprint -->
+	<link name="world" />
+	<link name="virtual_link1" />
+	<link name="virtual_link2" />
+	<joint name="odom_x" type="prismatic">
+		<origin xyz="0 0 0" rpy="0 0 0"/>
+		<parent link="world"/>
+		<child link="virtual_link1"/>
+	</joint>
+	<joint name="odom_y" type="prismatic">
+		<origin xyz="0 0 0" rpy="0 0 0"/>
+		<parent link="virtual_link1"/>
+		<child link="virtual_link2"/>
+	</joint>
+	<joint name="odom_r" type="prismatic">
+		<origin xyz="0 0 0" rpy="0 0 0"/>
+		<parent link="virtual_link2"/>
+		<child link="summit_xl_base_footprint"/>
+	</joint>
 	<!-- Import summit XL wheels -->
 	<xacro:include filename="$(find summit_xl_description)/urdf/wheels/omni_wheel.urdf.xacro" />
