Commit message: combined_moman.launch now works with gazebo

File: catkin_ws/src/summit_xl_common/summit_xl_description/robots/moman.urdf.xacro (robot description, xacro)
@@ -4,33 +4,6 @@
 	<!-- Imported elements -->
 	<!-- ***************** -->
-	<!-- First we import all posible elements defined in the urdf.xacro files. All these elements
-	are defined as macro:xacros -->
 	<!-- Import summit XL base elements -->
 	<xacro:include filename="$(find summit_xl_description)/urdf/bases/summit_xls_base.urdf.xacro" />
-	<!-- Define the joint between world and base_footprint -->
-	<link name="odom" />
-	<link name="virtual_link1" />
-	<link name="virtual_link2" />
-	<joint name="odom_x" type="prismatic">
-		<origin xyz="0 0 0" rpy="0 0 0"/>
-		<parent link="odom"/>
-		<child link="virtual_link1"/>
-        <axis xyz="1 0 0"/>
-        <limit effort="1000" lower="-10" upper="10" velocity="0.5"/>
-	</joint>
-	<joint name="odom_y" type="prismatic">
-		<origin xyz="0 0 0" rpy="0 0 0"/>
-		<parent link="virtual_link1"/>
-		<child link="virtual_link2"/>
-        <axis xyz="0 1 0"/>
-        <limit effort="1000" lower="-10" upper="10" velocity="0.5"/>
-	</joint>
-	<joint name="odom_r" type="revolute">
-		<origin xyz="0 0 0" rpy="0 0 0"/>
-		<parent link="virtual_link2"/>
-		<child link="summit_xl_base_footprint"/>
-        <axis xyz="0 0 1"/>
-        <limit effort="1000" lower="-3.14" upper="3.14" velocity="0.5"/>
-	</joint>
 	<!-- Import summit XL wheels -->
 	<xacro:include filename="$(find summit_xl_description)/urdf/wheels/omni_wheel.urdf.xacro" />
@@ -80,12 +53,4 @@
 	<!-- Name for this robot -->
 	<xacro:arg name="arm_id" default="panda" />
-	<!-- Should a franka_gripper be mounted at the flange?" -->
-	<xacro:arg name="hand" default="false" />
-	<!-- Positional offset between $(arm_id)_hand -> $(arm_id)_hand_tcp [m]. Only used when
-	hand:=true -->
-	<xacro:arg name="tcp_xyz" default="0 0 0.1034" />
-	<!-- Rotational offset between $(arm_id)_hand -> $(arm_id)_hand_tcp [rad]. Only used when
-	hand:=true -->
-	<xacro:arg name="tcp_rpy" default="0 0 0" />
 	<!-- Is the robot being simulated in gazebo?" -->
 	<xacro:arg name="gazebo" default="true" />
@@ -110,6 +75,4 @@
 		<!-- Robots Elements -->
 		<!-- *************** -->
-		<!-- Here we create the robot elements using the xacro:macros imported at the beggining of
-		this file -->
 		<!-- Summit XL base -->
 		<xacro:summit_xls_base prefix="$(arg prefix)" publish_bf="true" hq="${hq}" />
@@ -146,14 +109,4 @@
 				rpy="0 ${-PI} ${-1/4*PI}" />
 		</xacro:sensor_sick_s300>
-		<!--xacro:sensor_axis_m5013
-		prefix="$(arg prefix)front_ptz_camera" parent="$(arg prefix)base_link">
-			<origin xyz="${front_ptz_camera_offset_x} ${front_ptz_camera_offset_y}
-		${front_ptz_camera_offset_z}" rpy="${-PI/2} 0 0"/>
-		</xacro:sensor_axis_m5013-->
-		<!--xacro:sensor_axis_m5013
-		prefix="$(arg prefix)rear_ptz_camera" parent="$(arg prefix)base_link">
-			<origin xyz="${rear_ptz_camera_offset_x} ${rear_ptz_camera_offset_y} ${rear_ptz_camera_offset_z}"
-		rpy="${-PI/2} 0 ${PI}"/>
-		</xacro:sensor_axis_m5013-->
 		<xacro:sensor_orbbec_astra prefix="$(arg prefix)front_rgbd_camera"
 			parent="$(arg prefix)base_link" prefix_topic="front_rgbd_camera">
@@ -162,22 +115,6 @@
 				rpy="0 0 0" />
 		</xacro:sensor_orbbec_astra>
-		<!--xacro:sensor_gps
-		prefix="$(arg prefix)gps" parent="$(arg prefix)base_link">
-			<origin xyz="${gps_offset_x} ${gps_offset_y} ${gps_offset_z}" rpy="0 0 0"/>
-		</xacro:sensor_gps-->
-		<!-- Instance ViperX 300s arm -->
-		<!-- <joint name="$(arg prefix)arm_base_joint" type="fixed">
-			<origin xyz="${arm_offset_x} ${arm_offset_y} ${arm_offset_z}"
-				rpy="${arm_offset_roll} ${arm_offset_pitch} ${arm_offset_yaw}" />
-			<parent link="$(arg prefix)base_link" />
-			<child link="$(arg prefix)arm_base_link" />
-			<axis xyz="0 0 0" />
-		</joint> -->
-		<!-- <xacro:vx300s base_parent="$(arg prefix)arm_base_link" prefix="$(arg prefix)arm_" /> -->
 		<xacro:franka_robot arm_id="$(arg arm_id)"
 			joint_limits="${xacro.load_yaml('$(find franka_description)/robots/panda/joint_limits.yaml')}"
-			hand="$(arg hand)"
-			tcp_xyz="$(arg tcp_xyz)"
-			tcp_rpy="$(arg tcp_rpy)"
 			gazebo="$(arg gazebo)"
 			parent="$(arg prefix)base_link"

File: catkin_ws/src/summit_xl_common/summit_xl_description/urdf/bases/summit_xls_base.urdf.xacro (robot description, xacro)
@@ -3,147 +3,224 @@
   <xacro:include filename="$(find summit_xl_description)/urdf/bases/summit_xl_base.gazebo.xacro" />
   <xacro:macro name="summit_xls_base" params="prefix publish_bf hq">
-  <!-- Robot mechanical and motor parameters -->
-  <xacro:property name="PI" value="3.1415926535897931"/>
-  <xacro:property name="wheel_radius" value="0.127" />
-	<!-- BASE FOOTPRINT -->
-	  <xacro:if value="${publish_bf}">
-		<link name="${prefix}base_footprint">
-		  <visual>
-			  <origin xyz="0 0 0" rpy="0 0 0" />
-			  <geometry>
-				 <box size="0.001 0.001 0.001" />
-			  </geometry>
-		  </visual>
-		</link>
-		<joint name="${prefix}base_footprint_joint" type="fixed">
-		  <origin xyz="0 0 ${wheel_radius}" rpy="0 0 0" /> <!-- ${wheel_radius} property must be defined inside wheel description -->
-		  <parent link="${prefix}base_footprint"/>
-		  <child link="${prefix}base_link" />
-		</joint>
-	  </xacro:if>
-  <!-- BASE_LINK -->
-  <link name="${prefix}base_link">
-    <inertial>
-      <mass value="125.0" />
-      <origin xyz="0 0 0" />
-      <inertia  ixx="1.391" ixy="0.004"  ixz="0.0"  iyy="6.853"  iyz="0.0"  izz="6.125" />
-    </inertial>
-    <visual>
-      <origin xyz="0 0 0" rpy="0 0 0" />
-      <xacro:if value="${hq}">
-      <geometry>
-      <mesh filename="package://summit_xl_description/meshes/bases/xls/summit_xls_chassis.stl"/>
-      </geometry>
-      </xacro:if>
-      <xacro:unless value="${hq}">
-      <geometry>
-      <mesh filename="package://summit_xl_description/meshes/bases/xls/summit_xls_chassis.dae"/>
-      </geometry>
-      </xacro:unless>
-      <material name="black">
-        <color rgba="0.0 0.0 0.0 1"/>
-      </material>
-    </visual>
-    <collision>
-       <origin xyz="0 0 0" rpy="0 0 0 " />
-       <geometry>
-         <mesh filename="package://summit_xl_description/meshes/bases/xls/summit_xls_chassis.dae"/>
-       </geometry>
-    </collision>
-  </link>
-  <gazebo reference="${prefix}base_link">
-    <material>Gazebo/Black</material>
-  </gazebo>
-  <!-- CHAPAS INOX TAPAS -->
-  <link name="${prefix}base_chapa">
-  <visual>
-    <origin xyz="0 0 0" rpy="0 0 0" />
-    <geometry>
-    <mesh filename="package://summit_xl_description/meshes/bases/xls/summit_xls_chapas_inox_tapas.stl"/>
-    </geometry>
-    <material name="darkgrey">
-      <color rgba="0.5 0.5 0.5 1"/>
-    </material>
-    </visual>
-  </link>
-  <joint name="${prefix}base_tapa_joint" type="fixed">
-    <origin xyz="0.0 0 0.38062" rpy="0 0 0" />
-    <parent link="${prefix}base_link"/>
-    <child link="${prefix}base_chapa" />
-  </joint>
-  <!-- LOGO ROBOTNIK IZQUIERDO -->
-  <link name="${prefix}base_logo_left">
-  <visual>
-    <origin xyz="0 0 0" rpy="0 0 0" />
-    <geometry>
-    <mesh filename="package://summit_xl_description/meshes/bases/xls/robotnik_logo_chasis.stl"/>
-    </geometry>
-    <material name="darkgrey">
-      <color rgba="0.5 0.5 0.5 1"/>
-    </material>
-    </visual>
-  </link>
-  <joint name="${prefix}base_logo_left_joint" type="fixed">
-    <origin xyz="0.0 0.28931 0.29062" rpy="0 0 0" />
-    <parent link="${prefix}base_link"/>
-    <child link="${prefix}base_logo_left" />
-  </joint>
-  <!-- LOGO ROBOTNIK DERECHO -->
-  <link name="${prefix}base_logo_right">
-  <visual>
-    <origin xyz="0 0 0" rpy="0 0 0" />
-    <geometry>
-    <mesh filename="package://summit_xl_description/meshes/bases/xls/robotnik_logo_chasis.stl"/>
-    </geometry>
-    <material name="darkgrey">
-      <color rgba="0.5 0.5 0.5 1"/>
-    </material>
-    </visual>
-  </link>
-  <joint name="${prefix}base_logo_right_joint" type="fixed">
-    <origin xyz="0.0 -0.28931 0.29062" rpy="0 0 ${PI}" />
-    <parent link="${prefix}base_link"/>
-    <child link="${prefix}base_logo_right" />
-  </joint>
-  <!-- LOGO ROBOTNIK FRONTAL -->
-  <link name="${prefix}base_logo_front">
-  <visual>
-    <origin xyz="0 0 0" rpy="0 0 0" />
-    <geometry>
-    <mesh filename="package://summit_xl_description/meshes/bases/xls/robotnik_logo_chasis.stl"/>
-    </geometry>
-    <material name="darkgrey">
-      <color rgba="0.5 0.5 0.5 1"/>
-    </material>
-    </visual>
-  </link>
-  <joint name="${prefix}base_logo_front_joint" type="fixed">
-    <origin xyz="0.345 0.0 0.0" rpy="0 0 ${-PI/2}" />
-    <parent link="${prefix}base_link"/>
-    <child link="${prefix}base_logo_front" />
-  </joint>
-  <!-- LOGO ROBOTNIK TRASERO -->
-  <link name="${prefix}base_logo_rear">
-  <visual>
-    <origin xyz="0 0 0" rpy="0 0 0" />
-    <geometry>
-    <mesh filename="package://summit_xl_description/meshes/bases/xls/robotnik_logo_chasis.stl"/>
-    </geometry>
-    <material name="darkgrey">
-      <color rgba="0.5 0.5 0.5 1"/>
-    </material>
-    </visual>
-  </link>
-  <joint name="${prefix}base_logo_rear_joint" type="fixed">
-    <origin xyz="-0.345 0.0 0.0" rpy="0 0 ${PI/2}" />
-    <parent link="${prefix}base_link"/>
-    <child link="${prefix}base_logo_rear" />
-  </joint>
-   <!-- DOCKING CONTACT -->
+    <!-- Robot mechanical and motor parameters -->
+    <xacro:property name="PI" value="3.1415926535897931" />
+    <xacro:property name="wheel_radius" value="0.127" />
+    <link name="world" />
+    <link name="odom">
+      <inertial>
+        <mass value="0.01" />
+        <inertia ixx="1" ixy="0" ixz="0" iyy="1" iyz="0" izz="1" />
+      </inertial>
+    </link>
+    <link name="virtual_link1">
+      <inertial>
+        <mass value="0.01" />
+        <inertia ixx="1" ixy="0" ixz="0" iyy="1" iyz="0" izz="1" />
+      </inertial>
+    </link>
+    <link name="virtual_link2">
+      <inertial>
+        <mass value="0.01" />
+        <inertia ixx="1" ixy="0" ixz="0" iyy="1" iyz="0" izz="1" />
+      </inertial>
+    </link>
+    <joint name="world_base" type="fixed">
+      <parent link="world" />
+      <child link="odom" />
+    </joint>
+    <joint name="odom_x" type="prismatic">
+      <parent link="odom" />
+      <child link="virtual_link1" />
+      <axis xyz="1 0 0" />
+      <limit effort="1000000" lower="-10" upper="10" velocity="1000000" />
+    </joint>
+    <transmission name="odom_x_trans">
+      <type>transmission_interface/SimpleTransmission</type>
+      <joint name="odom_x">
+        <hardwareInterface>hardware_interface/EffortJointInterface</hardwareInterface>
+      </joint>
+      <actuator name="odom_x_motor">
+        <hardwareInterface>hardware_interface/EffortJointInterface</hardwareInterface>
+        <mechanicalReduction>1</mechanicalReduction>
+      </actuator>
+    </transmission>
+    <joint name="odom_y" type="prismatic">
+      <parent link="virtual_link1" />
+      <child link="virtual_link2" />
+      <axis xyz="0 1 0" />
+      <limit effort="1000000" lower="-10" upper="10" velocity="1000000" />
+    </joint>
+    <transmission name="odom_y_trans">
+      <type>transmission_interface/SimpleTransmission</type>
+      <joint name="odom_y">
+        <hardwareInterface>hardware_interface/EffortJointInterface</hardwareInterface>
+      </joint>
+      <actuator name="odom_y_motor">
+        <hardwareInterface>hardware_interface/EffortJointInterface</hardwareInterface>
+        <mechanicalReduction>1</mechanicalReduction>
+      </actuator>
+    </transmission>
+    <gazebo reference="odom_r">
+      <!-- Needed for ODE to output external wrenches on joints -->
+      <provideFeedback>true</provideFeedback>
+    </gazebo>
+    <joint name="odom_r" type="revolute">
+      <parent link="virtual_link2" />
+      <child link="${prefix}base_footprint" />
+      <axis xyz="0 0 1" />
+      <limit effort="1000" lower="-3.14" upper="3.14" velocity="100" />
+    </joint>
+    <transmission name="odom_r_transmission">
+      <type>transmission_interface/SimpleTransmission</type>
+      <joint name="odom_r">
+        <hardwareInterface>hardware_interface/EffortJointInterface</hardwareInterface>
+      </joint>
+      <actuator name="odom_r_motor">
+        <hardwareInterface>hardware_interface/EffortJointInterface</hardwareInterface>
+        <mechanicalReduction>1</mechanicalReduction>
+      </actuator>
+    </transmission>
+    <!-- BASE FOOTPRINT -->
+    <xacro:if value="${publish_bf}">
+      <link name="${prefix}base_footprint">
+        <visual>
+          <origin xyz="0 0 0" rpy="0 0 0" />
+          <geometry>
+            <box size="0.001 0.001 0.001" />
+          </geometry>
+        </visual>
+      </link>
+      <joint name="${prefix}base_footprint_joint" type="fixed">
+        <origin xyz="0 0 ${wheel_radius}" rpy="0 0 0" /> <!-- ${wheel_radius} property must be
+        defined inside wheel description -->
+        <parent link="${prefix}base_footprint" />
+        <child link="${prefix}base_link" />
+      </joint>
+    </xacro:if>
+    <!-- BASE_LINK -->
+    <link name="${prefix}base_link">
+      <inertial>
+        <mass value="125.0" />
+        <origin xyz="0 0 0" />
+        <inertia ixx="1.391" ixy="0.004" ixz="0.0" iyy="6.853" iyz="0.0" izz="6.125" />
+      </inertial>
+      <visual>
+        <origin xyz="0 0 0" rpy="0 0 0" />
+        <xacro:if value="${hq}">
+          <geometry>
+            <mesh filename="package://summit_xl_description/meshes/bases/xls/summit_xls_chassis.stl" />
+          </geometry>
+        </xacro:if>
+        <xacro:unless value="${hq}">
+          <geometry>
+            <mesh filename="package://summit_xl_description/meshes/bases/xls/summit_xls_chassis.dae" />
+          </geometry>
+        </xacro:unless>
+        <material name="black">
+          <color rgba="0.0 0.0 0.0 1" />
+        </material>
+      </visual>
+      <collision>
+        <origin xyz="0 0 0" rpy="0 0 0 " />
+        <geometry>
+          <mesh filename="package://summit_xl_description/meshes/bases/xls/summit_xls_chassis.dae" />
+        </geometry>
+      </collision>
+    </link>
+    <gazebo reference="${prefix}base_link">
+      <material>Gazebo/Black</material>
+    </gazebo>
+    <!-- CHAPAS INOX TAPAS -->
+    <link name="${prefix}base_chapa">
+      <visual>
+        <origin xyz="0 0 0" rpy="0 0 0" />
+        <geometry>
+          <mesh
+            filename="package://summit_xl_description/meshes/bases/xls/summit_xls_chapas_inox_tapas.stl" />
+        </geometry>
+        <material name="darkgrey">
+          <color rgba="0.5 0.5 0.5 1" />
+        </material>
+      </visual>
+    </link>
+    <joint name="${prefix}base_tapa_joint" type="fixed">
+      <origin xyz="0.0 0 0.38062" rpy="0 0 0" />
+      <parent link="${prefix}base_link" />
+      <child link="${prefix}base_chapa" />
+    </joint>
+    <!-- LOGO ROBOTNIK IZQUIERDO -->
+    <link name="${prefix}base_logo_left">
+      <visual>
+        <origin xyz="0 0 0" rpy="0 0 0" />
+        <geometry>
+          <mesh filename="package://summit_xl_description/meshes/bases/xls/robotnik_logo_chasis.stl" />
+        </geometry>
+        <material name="darkgrey">
+          <color rgba="0.5 0.5 0.5 1" />
+        </material>
+      </visual>
+    </link>
+    <joint name="${prefix}base_logo_left_joint" type="fixed">
+      <origin xyz="0.0 0.28931 0.29062" rpy="0 0 0" />
+      <parent link="${prefix}base_link" />
+      <child link="${prefix}base_logo_left" />
+    </joint>
+    <!-- LOGO ROBOTNIK DERECHO -->
+    <link name="${prefix}base_logo_right">
+      <visual>
+        <origin xyz="0 0 0" rpy="0 0 0" />
+        <geometry>
+          <mesh filename="package://summit_xl_description/meshes/bases/xls/robotnik_logo_chasis.stl" />
+        </geometry>
+        <material name="darkgrey">
+          <color rgba="0.5 0.5 0.5 1" />
+        </material>
+      </visual>
+    </link>
+    <joint name="${prefix}base_logo_right_joint" type="fixed">
+      <origin xyz="0.0 -0.28931 0.29062" rpy="0 0 ${PI}" />
+      <parent link="${prefix}base_link" />
+      <child link="${prefix}base_logo_right" />
+    </joint>
+    <!-- LOGO ROBOTNIK FRONTAL -->
+    <link name="${prefix}base_logo_front">
+      <visual>
+        <origin xyz="0 0 0" rpy="0 0 0" />
+        <geometry>
+          <mesh filename="package://summit_xl_description/meshes/bases/xls/robotnik_logo_chasis.stl" />
+        </geometry>
+        <material name="darkgrey">
+          <color rgba="0.5 0.5 0.5 1" />
+        </material>
+      </visual>
+    </link>
+    <joint name="${prefix}base_logo_front_joint" type="fixed">
+      <origin xyz="0.345 0.0 0.0" rpy="0 0 ${-PI/2}" />
+      <parent link="${prefix}base_link" />
+      <child link="${prefix}base_logo_front" />
+    </joint>
+    <!-- LOGO ROBOTNIK TRASERO -->
+    <link name="${prefix}base_logo_rear">
+      <visual>
+        <origin xyz="0 0 0" rpy="0 0 0" />
+        <geometry>
+          <mesh filename="package://summit_xl_description/meshes/bases/xls/robotnik_logo_chasis.stl" />
+        </geometry>
+        <material name="darkgrey">
+          <color rgba="0.5 0.5 0.5 1" />
+        </material>
+      </visual>
+    </link>
+    <joint name="${prefix}base_logo_rear_joint" type="fixed">
+      <origin xyz="-0.345 0.0 0.0" rpy="0 0 ${PI/2}" />
+      <parent link="${prefix}base_link" />
+      <child link="${prefix}base_logo_rear" />
+    </joint>
+    <!-- DOCKING CONTACT -->
     <link name="${prefix}base_docking_contact">
     </link>
     <joint name="${prefix}base_docking_joint" type="fixed">
       <origin xyz="0.35 0 0.09" rpy="0 0 0" />
-      <parent link="${prefix}base_link"/>
+      <parent link="${prefix}base_link" />
       <child link="${prefix}base_docking_contact" />
     </joint>
