Commit message: cleaned up and added service

File: catkin_ws/src/summit_xl_common/summit_xl_description/robots/panda.urdf (robot description, URDF)
Before this commit: robot summit_xl, 39 links, 38 joints
Links:
- added link odom, mass 0.01
- added link virtual_link1, mass 0.01
- added link virtual_link2, mass 0.01
- added link world
Joints:
- added joint odom_r: type revolute, parent virtual_link2, child summit_xl_base_footprint, axis 0 0 1, limit lower=-3.14 upper=3.14 effort=1000 velocity=100
- added joint odom_x: type prismatic, parent odom, child virtual_link1, axis 1 0 0, limit lower=-10 upper=10 effort=1000000 velocity=1000000
- added joint odom_y: type prismatic, parent virtual_link1, child virtual_link2, axis 0 1 0, limit lower=-10 upper=10 effort=1000000 velocity=1000000
- added joint world_base: type fixed, parent world, child odom

File: catkin_ws/src/summit_xl_common/summit_xl_description/urdf/bases/summit_xl_base.gazebo.xacro (robot description, xacro)
@@ -4,5 +4,5 @@
 	<xacro:macro name="ros_control">
 		<gazebo>
-			<plugin name="ros_control" filename="libgazebo_ros_control.so">
+			<plugin name="ros_control" filename="libgazeboa_ros_control.so">
 				<robotParam>robot_description</robotParam>
 				<controlPeriod>0.001</controlPeriod>
