Commit message: lgtm

File: catkin_ws/src/summit_xl_common/summit_xl_description/urdf/arms/franka/franka_robot.xacro (robot description, xacro)
@@ -21,5 +21,5 @@
     <!-- Define additional Gazebo tags -->
     <!-- <xacro:if value="${gazebo}"> -->
-    <xacro:if value="false">
+    <xacro:if value="${gazebo}">
       <!-- PERHAPS COMMENT THIS OUT IT MIGHT BE DUPLICATING THE ROBOT GIVING THE FOLLOWING ERROR -->
       <!-- Warning [Model.cc:216] Non-unique name[koala_joint7] detected 2 times in XML children of

File: catkin_ws/src/summit_xl_common/summit_xl_description/urdf/bases/summit_xl_base.gazebo.xacro (robot description, xacro)
@@ -1,38 +1,39 @@
 <?xml version="1.0"?>
 <robot xmlns:xacro="http://wiki.ros.org/xacro">
-  <!-- ros control plugin -->
-  <xacro:macro name="ros_control">
-    <gazebo>
-      <plugin name="ros_control" filename="libgazebo_ros_control.so">
-		    <robotParam>robot_description</robotParam>
-        <controlPeriod>0.001</controlPeriod>
-	      <robotSimType>gazebo_ros_control/DefaultRobotHWSim</robotSimType>
-		    <legacyModeNS>true</legacyModeNS>
-      </plugin>
-    </gazebo>
+	<!-- ros control plugin -->
+	<xacro:macro name="ros_control">
+		<gazebo>
+			<plugin name="ros_control" filename="libgazebo_ros_control.so">
+				<robotParam>robot_description</robotParam>
+				<controlPeriod>0.001</controlPeriod>
+				<robotSimType>gazebo_ros_control/DefaultRobotHWSim</robotSimType>
+				<legacyModeNS>true</legacyModeNS>
+			</plugin>
+		</gazebo>
 	</xacro:macro>
 	<!-- skid steering plugin -->
 	<xacro:macro name="skid_steering" params="prefix publish_tf">
-    <gazebo>
-      <plugin name="skid_steer_drive_controller" filename="libgazebo_ros_skid_steer_drive.so">
-			<!--<robotNamespace>/summit_xl</robotNamespace>-->
-		    <updateRate>50.0</updateRate>
-		    <leftFrontJoint>${prefix}front_left_wheel_joint</leftFrontJoint>
-		    <rightFrontJoint>${prefix}front_right_wheel_joint</rightFrontJoint>
-		    <leftRearJoint>${prefix}back_left_wheel_joint</leftRearJoint>
-		    <rightRearJoint>${prefix}back_right_wheel_joint</rightRearJoint>
-		    <!-- wheelSeparation>0.566</wheelSeparation --> <!-- real parameter value -->
-		    <wheelSeparation>0.462</wheelSeparation> <!-- works a bit better in Gazebo -->
-		    <wheelDiameter>0.22</wheelDiameter>
-		    <robotBaseFrame>${prefix}base_footprint</robotBaseFrame>
-		    <torque>50</torque>
-		    <commandTopic>robotnik_base_control/cmd_vel</commandTopic>
-		    <odometryTopic>robotnik_base_control/odom</odometryTopic>
-		    <odometryFrame>${prefix}odom</odometryFrame>
-		    <broadcastTF>${publish_tf}</broadcastTF>
-      </plugin>
-    </gazebo>
-  </xacro:macro>
-  <xacro:macro name="omni_steering" params="prefix publish_tf force_based:=false">
+		<gazebo>
+			<plugin name="skid_steer_drive_controller" filename="libgazebo_ros_skid_steer_drive.so">
+				<!--<robotNamespace>/summit_xl</robotNamespace>-->
+				<updateRate>50.0</updateRate>
+				<leftFrontJoint>${prefix}front_left_wheel_joint</leftFrontJoint>
+				<rightFrontJoint>${prefix}front_right_wheel_joint</rightFrontJoint>
+				<leftRearJoint>${prefix}back_left_wheel_joint</leftRearJoint>
+				<rightRearJoint>${prefix}back_right_wheel_joint</rightRearJoint>
+				<!-- wheelSeparation>0.566</wheelSeparation --> <!-- real parameter
+				value -->
+				<wheelSeparation>0.462</wheelSeparation> <!-- works a bit better in Gazebo -->
+				<wheelDiameter>0.22</wheelDiameter>
+				<robotBaseFrame>${prefix}base_footprint</robotBaseFrame>
+				<torque>50</torque>
+				<commandTopic>robotnik_base_control/cmd_vel</commandTopic>
+				<odometryTopic>robotnik_base_control/odom</odometryTopic>
+				<odometryFrame>${prefix}odom</odometryFrame>
+				<broadcastTF>${publish_tf}</broadcastTF>
+			</plugin>
+		</gazebo>
+	</xacro:macro>
+	<xacro:macro name="omni_steering" params="prefix publish_tf force_based:=false">
 		<xacro:if value="${force_based}">
 			<gazebo>
@@ -54,16 +55,16 @@
 			<gazebo>
 				<plugin name="omni_steering" filename="libgazebo_ros_planar_move.so">
-				<commandTopic>robotnik_base_control/cmd_vel</commandTopic>
-				<odometryTopic>robotnik_base_control/odom</odometryTopic>
-				<odometryFrame>${prefix}odom</odometryFrame>
-				<odometryRate>50.0</odometryRate>
-				<robotBaseFrame>${prefix}base_footprint</robotBaseFrame>
-				<publishTF>${publish_tf}</publishTF>
-				<enableYAxis>true</enableYAxis>
+					<commandTopic>robotnik_base_control/cmd_vel</commandTopic>
+					<odometryTopic>robotnik_base_control/odom</odometryTopic>
+					<odometryFrame>${prefix}odom</odometryFrame>
+					<odometryRate>50.0</odometryRate>
+					<robotBaseFrame>${prefix}base_footprint</robotBaseFrame>
+					<publishTF>${publish_tf}</publishTF>
+					<enableYAxis>true</enableYAxis>
 				</plugin>
 			</gazebo>
 		</xacro:unless>
-  </xacro:macro>
-  	<xacro:macro name="skid_steering" params="prefix publish_tf force_based">
+	</xacro:macro>
+	<xacro:macro name="skid_steering" params="prefix publish_tf force_based">
 		<xacro:if value="${force_based}">
 			<gazebo>
@@ -82,36 +83,36 @@
 			</gazebo>
 		</xacro:if>
-	  	<xacro:unless value="${force_based}">
+		<xacro:unless value="${force_based}">
 			<gazebo>
 				<plugin name="skid_steering" filename="libgazebo_ros_planar_move.so">
+					<commandTopic>robotnik_base_control/cmd_vel</commandTopic>
+					<odometryTopic>robotnik_base_control/odom</odometryTopic>
+					<odometryFrame>${prefix}odom</odometryFrame>
+					<odometryRate>50.0</odometryRate>
+					<robotBaseFrame>${prefix}base_footprint</robotBaseFrame>
+					<publishTF>${publish_tf}</publishTF>
+					<enableYAxis>false</enableYAxis>
+				</plugin>
+			</gazebo>
+		</xacro:unless>
+	</xacro:macro>
+	<xacro:macro name="ros_force_based_move" params="publish_tf prefix">
+		<gazebo>
+			<plugin name="ros_force_based_move" filename="librobotnik_force_based_move.so">
 				<commandTopic>robotnik_base_control/cmd_vel</commandTopic>
 				<odometryTopic>robotnik_base_control/odom</odometryTopic>
 				<odometryFrame>${prefix}odom</odometryFrame>
+				<yaw_velocity_p_gain>10000.0</yaw_velocity_p_gain>
+				<x_velocity_p_gain>10000.0</x_velocity_p_gain>
+				<y_velocity_p_gain>10000.0</y_velocity_p_gain>
+				<robotBaseFrame>${prefix}base_footprint</robotBaseFrame>
+				<commandWatchdog>1</commandWatchdog>
 				<odometryRate>50.0</odometryRate>
-				<robotBaseFrame>${prefix}base_footprint</robotBaseFrame>
-				<publishTF>${publish_tf}</publishTF>
-				<enableYAxis>false</enableYAxis>
-				</plugin>
-			</gazebo>
-		</xacro:unless>
-  	</xacro:macro>
-  <xacro:macro name="ros_force_based_move" params="publish_tf prefix">
-	  <gazebo>
-		 <plugin name="ros_force_based_move" filename="librobotnik_force_based_move.so">
-			 <commandTopic>robotnik_base_control/cmd_vel</commandTopic>
-			 <odometryTopic>robotnik_base_control/odom</odometryTopic>
-	         <odometryFrame>${prefix}odom</odometryFrame>
-			 <yaw_velocity_p_gain>10000.0</yaw_velocity_p_gain>
-			 <x_velocity_p_gain>10000.0</x_velocity_p_gain>
-			 <y_velocity_p_gain>10000.0</y_velocity_p_gain>
-			 <robotBaseFrame>${prefix}base_footprint</robotBaseFrame>
-			 <commandWatchdog>1</commandWatchdog>
-			 <odometryRate>50.0</odometryRate>
-			 <publishOdometryTf>${publish_tf}</publishOdometryTf>
-		 </plugin>
-	  </gazebo>
-  </xacro:macro>
-  <gazebo reference="base_footprint">
-    <material>Gazebo/Green</material>
-  </gazebo>
+				<publishOdometryTf>${publish_tf}</publishOdometryTf>
+			</plugin>
+		</gazebo>
+	</xacro:macro>
+	<gazebo reference="base_footprint">
+		<material>Gazebo/Green</material>
+	</gazebo>
 </robot>

Commit message: some clean-up

File: catkin_ws/src/summit_xl_common/summit_xl_description/urdf/arms/franka/franka_robot.xacro (robot description, xacro)
@@ -2,5 +2,5 @@
 <robot xmlns:xacro="http://www.ros.org/wiki/xacro">
   <xacro:macro name="franka_robot"
-    params="arm_id joint_limits parent:='world' xyz:='0 0 0' rpy:='0 0 0' hand:=false gazebo:=false tcp_xyz:='0 0 0.1034' tcp_rpy='0 0 0'">
+    params="arm_id joint_limits parent:='world' xyz:='0 0 0' rpy:='0 0 0'  gazebo:=false ">
     <xacro:include filename="$(find franka_description)/robots/common/utils.xacro" />
     <xacro:include filename="$(find franka_description)/robots/common/franka_arm.xacro" />

File: catkin_ws/src/summit_xl_common/summit_xl_description/urdf/bases/summit_xls_base.urdf.xacro (robot description, xacro)
@@ -3,147 +3,177 @@
   <xacro:include filename="$(find summit_xl_description)/urdf/bases/summit_xl_base.gazebo.xacro" />
   <xacro:macro name="summit_xls_base" params="prefix publish_bf hq">
-  <!-- Robot mechanical and motor parameters -->
-  <xacro:property name="PI" value="3.1415926535897931"/>
-  <xacro:property name="wheel_radius" value="0.127" />
-	<!-- BASE FOOTPRINT -->
-	  <xacro:if value="${publish_bf}">
-		<link name="${prefix}base_footprint">
-		  <visual>
-			  <origin xyz="0 0 0" rpy="0 0 0" />
-			  <geometry>
-				 <box size="0.001 0.001 0.001" />
-			  </geometry>
-		  </visual>
-		</link>
-		<joint name="${prefix}base_footprint_joint" type="fixed">
-		  <origin xyz="0 0 ${wheel_radius}" rpy="0 0 0" /> <!-- ${wheel_radius} property must be defined inside wheel description -->
-		  <parent link="${prefix}base_footprint"/>
-		  <child link="${prefix}base_link" />
-		</joint>
-	  </xacro:if>
-  <!-- BASE_LINK -->
-  <link name="${prefix}base_link">
-    <inertial>
-      <mass value="125.0" />
-      <origin xyz="0 0 0" />
-      <inertia  ixx="1.391" ixy="0.004"  ixz="0.0"  iyy="6.853"  iyz="0.0"  izz="6.125" />
-    </inertial>
-    <visual>
-      <origin xyz="0 0 0" rpy="0 0 0" />
-      <xacro:if value="${hq}">
-      <geometry>
-      <mesh filename="package://summit_xl_description/meshes/bases/xls/summit_xls_chassis.stl"/>
-      </geometry>
-      </xacro:if>
-      <xacro:unless value="${hq}">
-      <geometry>
-      <mesh filename="package://summit_xl_description/meshes/bases/xls/summit_xls_chassis.dae"/>
-      </geometry>
-      </xacro:unless>
-      <material name="black">
-        <color rgba="0.0 0.0 0.0 1"/>
-      </material>
-    </visual>
-    <collision>
-       <origin xyz="0 0 0" rpy="0 0 0 " />
-       <geometry>
-         <mesh filename="package://summit_xl_description/meshes/bases/xls/summit_xls_chassis.dae"/>
-       </geometry>
-    </collision>
-  </link>
-  <gazebo reference="${prefix}base_link">
-    <material>Gazebo/Black</material>
-  </gazebo>
-  <!-- CHAPAS INOX TAPAS -->
-  <link name="${prefix}base_chapa">
-  <visual>
-    <origin xyz="0 0 0" rpy="0 0 0" />
-    <geometry>
-    <mesh filename="package://summit_xl_description/meshes/bases/xls/summit_xls_chapas_inox_tapas.stl"/>
-    </geometry>
-    <material name="darkgrey">
-      <color rgba="0.5 0.5 0.5 1"/>
-    </material>
-    </visual>
-  </link>
-  <joint name="${prefix}base_tapa_joint" type="fixed">
-    <origin xyz="0.0 0 0.38062" rpy="0 0 0" />
-    <parent link="${prefix}base_link"/>
-    <child link="${prefix}base_chapa" />
-  </joint>
-  <!-- LOGO ROBOTNIK IZQUIERDO -->
-  <link name="${prefix}base_logo_left">
-  <visual>
-    <origin xyz="0 0 0" rpy="0 0 0" />
-    <geometry>
-    <mesh filename="package://summit_xl_description/meshes/bases/xls/robotnik_logo_chasis.stl"/>
-    </geometry>
-    <material name="darkgrey">
-      <color rgba="0.5 0.5 0.5 1"/>
-    </material>
-    </visual>
-  </link>
-  <joint name="${prefix}base_logo_left_joint" type="fixed">
-    <origin xyz="0.0 0.28931 0.29062" rpy="0 0 0" />
-    <parent link="${prefix}base_link"/>
-    <child link="${prefix}base_logo_left" />
-  </joint>
-  <!-- LOGO ROBOTNIK DERECHO -->
-  <link name="${prefix}base_logo_right">
-  <visual>
-    <origin xyz="0 0 0" rpy="0 0 0" />
-    <geometry>
-    <mesh filename="package://summit_xl_description/meshes/bases/xls/robotnik_logo_chasis.stl"/>
-    </geometry>
-    <material name="darkgrey">
-      <color rgba="0.5 0.5 0.5 1"/>
-    </material>
-    </visual>
-  </link>
-  <joint name="${prefix}base_logo_right_joint" type="fixed">
-    <origin xyz="0.0 -0.28931 0.29062" rpy="0 0 ${PI}" />
-    <parent link="${prefix}base_link"/>
-    <child link="${prefix}base_logo_right" />
-  </joint>
-  <!-- LOGO ROBOTNIK FRONTAL -->
-  <link name="${prefix}base_logo_front">
-  <visual>
-    <origin xyz="0 0 0" rpy="0 0 0" />
-    <geometry>
-    <mesh filename="package://summit_xl_description/meshes/bases/xls/robotnik_logo_chasis.stl"/>
-    </geometry>
-    <material name="darkgrey">
-      <color rgba="0.5 0.5 0.5 1"/>
-    </material>
-    </visual>
-  </link>
-  <joint name="${prefix}base_logo_front_joint" type="fixed">
-    <origin xyz="0.345 0.0 0.0" rpy="0 0 ${-PI/2}" />
-    <parent link="${prefix}base_link"/>
-    <child link="${prefix}base_logo_front" />
-  </joint>
-  <!-- LOGO ROBOTNIK TRASERO -->
-  <link name="${prefix}base_logo_rear">
-  <visual>
-    <origin xyz="0 0 0" rpy="0 0 0" />
-    <geometry>
-    <mesh filename="package://summit_xl_description/meshes/bases/xls/robotnik_logo_chasis.stl"/>
-    </geometry>
-    <material name="darkgrey">
-      <color rgba="0.5 0.5 0.5 1"/>
-    </material>
-    </visual>
-  </link>
-  <joint name="${prefix}base_logo_rear_joint" type="fixed">
-    <origin xyz="-0.345 0.0 0.0" rpy="0 0 ${PI/2}" />
-    <parent link="${prefix}base_link"/>
-    <child link="${prefix}base_logo_rear" />
-  </joint>
-   <!-- DOCKING CONTACT -->
+    <!-- Robot mechanical and motor parameters -->
+    <xacro:property name="PI" value="3.1415926535897931" />
+    <xacro:property name="wheel_radius" value="0.127" />
+    <!-- Define the joint between world and base_footprint -->
+    <link name="dummy" />
+    <link name="virtual_link">
+      <inertial>
+        <mass value="0.01" />
+        <inertia ixx="1" ixy="0" ixz="0" iyy="1" iyz="0" izz="1" />
+      </inertial>
+    </link>
+    <joint name="world_base" type="fixed">
+      <parent link="dummy" />
+      <child link="virtual_link" />
+    </joint>
+    <joint name="odom_r" type="revolute">
+      <parent link="virtual_link" />
+      <child link="${prefix}base_footprint" />
+      <axis xyz="0 0 1" />
+      <limit effort="1000" lower="-3.14" upper="3.14" velocity="0.5" />
+    </joint>
+    <transmission name="odom_r_transmission">
+      <type>transmission_interface/SimpleTransmission</type>
+      <joint name="odom_r">
+        <hardwareInterface>hardware_interface/EffortJointInterface</hardwareInterface>
+      </joint>
+      <actuator name="odom_r_motor">
+        <hardwareInterface>hardware_interface/EffortJointInterface</hardwareInterface>
+        <mechanicalReduction>1</mechanicalReduction>
+      </actuator>
+    </transmission>
+    <!-- BASE FOOTPRINT -->
+    <xacro:if value="${publish_bf}">
+      <link name="${prefix}base_footprint">
+        <visual>
+          <origin xyz="0 0 0" rpy="0 0 0" />
+          <geometry>
+            <box size="0.001 0.001 0.001" />
+          </geometry>
+        </visual>
+      </link>
+      <joint name="${prefix}base_footprint_joint" type="fixed">
+        <origin xyz="0 0 ${wheel_radius}" rpy="0 0 0" /> <!-- ${wheel_radius} property must be
+        defined inside wheel description -->
+        <parent link="${prefix}base_footprint" />
+        <child link="${prefix}base_link" />
+      </joint>
+    </xacro:if>
+    <!-- BASE_LINK -->
+    <link name="${prefix}base_link">
+      <inertial>
+        <mass value="125.0" />
+        <origin xyz="0 0 0" />
+        <inertia ixx="1.391" ixy="0.004" ixz="0.0" iyy="6.853" iyz="0.0" izz="6.125" />
+      </inertial>
+      <visual>
+        <origin xyz="0 0 0" rpy="0 0 0" />
+        <xacro:if value="${hq}">
+          <geometry>
+            <mesh filename="package://summit_xl_description/meshes/bases/xls/summit_xls_chassis.stl" />
+          </geometry>
+        </xacro:if>
+        <xacro:unless value="${hq}">
+          <geometry>
+            <mesh filename="package://summit_xl_description/meshes/bases/xls/summit_xls_chassis.dae" />
+          </geometry>
+        </xacro:unless>
+        <material name="black">
+          <color rgba="0.0 0.0 0.0 1" />
+        </material>
+      </visual>
+      <collision>
+        <origin xyz="0 0 0" rpy="0 0 0 " />
+        <geometry>
+          <mesh filename="package://summit_xl_description/meshes/bases/xls/summit_xls_chassis.dae" />
+        </geometry>
+      </collision>
+    </link>
+    <gazebo reference="${prefix}base_link">
+      <material>Gazebo/Black</material>
+    </gazebo>
+    <!-- CHAPAS INOX TAPAS -->
+    <link name="${prefix}base_chapa">
+      <visual>
+        <origin xyz="0 0 0" rpy="0 0 0" />
+        <geometry>
+          <mesh
+            filename="package://summit_xl_description/meshes/bases/xls/summit_xls_chapas_inox_tapas.stl" />
+        </geometry>
+        <material name="darkgrey">
+          <color rgba="0.5 0.5 0.5 1" />
+        </material>
+      </visual>
+    </link>
+    <joint name="${prefix}base_tapa_joint" type="fixed">
+      <origin xyz="0.0 0 0.38062" rpy="0 0 0" />
+      <parent link="${prefix}base_link" />
+      <child link="${prefix}base_chapa" />
+    </joint>
+    <!-- LOGO ROBOTNIK IZQUIERDO -->
+    <link name="${prefix}base_logo_left">
+      <visual>
+        <origin xyz="0 0 0" rpy="0 0 0" />
+        <geometry>
+          <mesh filename="package://summit_xl_description/meshes/bases/xls/robotnik_logo_chasis.stl" />
+        </geometry>
+        <material name="darkgrey">
+          <color rgba="0.5 0.5 0.5 1" />
+        </material>
+      </visual>
+    </link>
+    <joint name="${prefix}base_logo_left_joint" type="fixed">
+      <origin xyz="0.0 0.28931 0.29062" rpy="0 0 0" />
+      <parent link="${prefix}base_link" />
+      <child link="${prefix}base_logo_left" />
+    </joint>
+    <!-- LOGO ROBOTNIK DERECHO -->
+    <link name="${prefix}base_logo_right">
+      <visual>
+        <origin xyz="0 0 0" rpy="0 0 0" />
+        <geometry>
+          <mesh filename="package://summit_xl_description/meshes/bases/xls/robotnik_logo_chasis.stl" />
+        </geometry>
+        <material name="darkgrey">
+          <color rgba="0.5 0.5 0.5 1" />
+        </material>
+      </visual>
+    </link>
+    <joint name="${prefix}base_logo_right_joint" type="fixed">
+      <origin xyz="0.0 -0.28931 0.29062" rpy="0 0 ${PI}" />
+      <parent link="${prefix}base_link" />
+      <child link="${prefix}base_logo_right" />
+    </joint>
+    <!-- LOGO ROBOTNIK FRONTAL -->
+    <link name="${prefix}base_logo_front">
+      <visual>
+        <origin xyz="0 0 0" rpy="0 0 0" />
+        <geometry>
+          <mesh filename="package://summit_xl_description/meshes/bases/xls/robotnik_logo_chasis.stl" />
+        </geometry>
+        <material name="darkgrey">
+          <color rgba="0.5 0.5 0.5 1" />
+        </material>
+      </visual>
+    </link>
+    <joint name="${prefix}base_logo_front_joint" type="fixed">
+      <origin xyz="0.345 0.0 0.0" rpy="0 0 ${-PI/2}" />
+      <parent link="${prefix}base_link" />
+      <child link="${prefix}base_logo_front" />
+    </joint>
+    <!-- LOGO ROBOTNIK TRASERO -->
+    <link name="${prefix}base_logo_rear">
+      <visual>
+        <origin xyz="0 0 0" rpy="0 0 0" />
+        <geometry>
+          <mesh filename="package://summit_xl_description/meshes/bases/xls/robotnik_logo_chasis.stl" />
+        </geometry>
+        <material name="darkgrey">
+          <color rgba="0.5 0.5 0.5 1" />
+        </material>
+      </visual>
+    </link>
+    <joint name="${prefix}base_logo_rear_joint" type="fixed">
+      <origin xyz="-0.345 0.0 0.0" rpy="0 0 ${PI/2}" />
+      <parent link="${prefix}base_link" />
+      <child link="${prefix}base_logo_rear" />
+    </joint>
+    <!-- DOCKING CONTACT -->
     <link name="${prefix}base_docking_contact">
     </link>
     <joint name="${prefix}base_docking_joint" type="fixed">
       <origin xyz="0.35 0 0.09" rpy="0 0 0" />
-      <parent link="${prefix}base_link"/>
+      <parent link="${prefix}base_link" />
       <child link="${prefix}base_docking_contact" />
     </joint>
