Commit message: Update

File: catkin_ws/src/moman_moveit_config/config/gazebo_summit_xl.urdf (robot description, URDF)
Before this commit: robot summit_xl, 42 links, 41 joints
Joints:
- joint odom_r: limit effort=1000 velocity=0.5 -> effort=1000 velocity=1
- joint odom_x: limit effort=1000 velocity=0.5 -> effort=1000 velocity=1
- joint odom_y: limit effort=1000 velocity=0.5 -> effort=1000 velocity=1
