Commit message: now all parts of the planar joints are actuated through moveit and into gazebo :D

File: catkin_ws/src/summit_xl_common/summit_xl_description/urdf/bases/summit_xls_base.urdf.xacro (robot description, xacro)
@@ -6,7 +6,6 @@
     <xacro:property name="PI" value="3.1415926535897931" />
     <xacro:property name="wheel_radius" value="0.127" />
-    <!-- Define the joint between world and base_footprint -->
-    <link name="dummy" />
-    <link name="virtual_link">
+    <link name="world" />
+    <link name="odom">
       <inertial>
         <mass value="0.01" />
@@ -14,13 +13,61 @@
       </inertial>
     </link>
+    <link name="virtual_link1">
+      <inertial>
+        <mass value="0.01" />
+        <inertia ixx="1" ixy="0" ixz="0" iyy="1" iyz="0" izz="1" />
+      </inertial>
+    </link>
+    <link name="virtual_link2">
+      <inertial>
+        <mass value="0.01" />
+        <inertia ixx="1" ixy="0" ixz="0" iyy="1" iyz="0" izz="1" />
+      </inertial>
+    </link>
     <joint name="world_base" type="fixed">
-      <parent link="dummy" />
-      <child link="virtual_link" />
-    </joint>
+      <parent link="world" />
+      <child link="odom" />
+    </joint>
+    <joint name="odom_x" type="prismatic">
+      <parent link="odom" />
+      <child link="virtual_link1" />
+      <axis xyz="1 0 0" />
+      <limit effort="1000000" lower="-10" upper="10" velocity="1000000" />
+    </joint>
+    <transmission name="odom_x_trans">
+      <type>transmission_interface/SimpleTransmission</type>
+      <joint name="odom_x">
+        <hardwareInterface>hardware_interface/EffortJointInterface</hardwareInterface>
+      </joint>
+      <actuator name="odom_x_motor">
+        <hardwareInterface>hardware_interface/EffortJointInterface</hardwareInterface>
+        <mechanicalReduction>1</mechanicalReduction>
+      </actuator>
+    </transmission>
+    <joint name="odom_y" type="prismatic">
+      <parent link="virtual_link1" />
+      <child link="virtual_link2" />
+      <axis xyz="0 1 0" />
+      <limit effort="1000000" lower="-10" upper="10" velocity="1000000" />
+    </joint>
+    <transmission name="odom_y_trans">
+      <type>transmission_interface/SimpleTransmission</type>
+      <joint name="odom_y">
+        <hardwareInterface>hardware_interface/EffortJointInterface</hardwareInterface>
+      </joint>
+      <actuator name="odom_y_motor">
+        <hardwareInterface>hardware_interface/EffortJointInterface</hardwareInterface>
+        <mechanicalReduction>1</mechanicalReduction>
+      </actuator>
+    </transmission>
+    <gazebo reference="odom_r">
+      <!-- Needed for ODE to output external wrenches on joints -->
+      <provideFeedback>true</provideFeedback>
+    </gazebo>
     <joint name="odom_r" type="revolute">
-      <parent link="virtual_link" />
+      <parent link="virtual_link2" />
       <child link="${prefix}base_footprint" />
       <axis xyz="0 0 1" />
-      <limit effort="1000" lower="-3.14" upper="3.14" velocity="0.5" />
+      <limit effort="1000" lower="-3.14" upper="3.14" velocity="100" />
     </joint>
     <transmission name="odom_r_transmission">

Commit message: post tracking commit

File: catkin_ws/src/summit_xl_common/summit_xl_description/urdf/bases/summit_xls_base.urdf.xacro (robot description, xacro)
@@ -65,9 +65,9 @@
       <provideFeedback>true</provideFeedback>
     </gazebo>
-    <joint name="odom_r" type="revolute">
+    <joint name="odom_r" type="continuous">
       <parent link="virtual_link2" />
       <child link="${prefix}base_footprint" />
       <axis xyz="0 0 1" />
-      <limit effort="1000" lower="-3.14" upper="3.14" velocity="100" />
+      <!-- <limit effort="1000" lower="-3.14" upper="3.14" velocity="100" /> -->
     </joint>
     <transmission name="odom_r_transmission">

Commit message: Large push with data from tests

File: catkin_ws/src/summit_xl_common/summit_xl_description/urdf/bases/summit_xls_base.urdf.xacro (robot description, xacro)
@@ -33,5 +33,5 @@
       <child link="virtual_link1" />
       <axis xyz="1 0 0" />
-      <limit effort="1000000" lower="-10" upper="10" velocity="1000000" />
+      <limit effort="1000000" lower="-50" upper="50" velocity="1000000" />
     </joint>
     <transmission name="odom_x_trans">
@@ -49,5 +49,5 @@
       <child link="virtual_link2" />
       <axis xyz="0 1 0" />
-      <limit effort="1000000" lower="-10" upper="10" velocity="1000000" />
+      <limit effort="1000000" lower="-50" upper="50" velocity="1000000" />
     </joint>
     <transmission name="odom_y_trans">
